File: RKD_01/RKD01_Top_L/RKD01_Top_L.kicad_pcb (KiCad board)
At the start: 2 copper layers, 164.3 x 102.4 mm, 42 parts, among them SW1 SW_Push, SW10 SW_Push, SW11 SW_Push, SW12 SW_Push, SW13 SW_Push, SW14 SW_Push, SW15 SW_Push, SW16 SW_Push, SW17 SW_Push, SW18 SW_Push, SW19 SW_Push, SW2 SW_Push, SW20 SW_Push, SW21 SW_Push, SW22 SW_Push, SW23 SW_Push, SW24 SW_Push, SW25 SW_Push, SW26 SW_Push, SW27 SW_Push, SW28 SW_Push, SW29 SW_Push, SW3 SW_Push, SW30 SW_Push, SW31 SW_Push, SW32 SW_Push, SW33 SW_Push, SW34 RotaryEncoder_Switch, SW4 SW_Push, SW5 SW_Push, SW6 SW_Push, SW66 SW_PUSH, SW7 SW_Push, SW8 SW_Push, SW9 SW_Push

Commit message: LeftTop最終生
Parts:
- removed SW66 (x2): SW_PUSH, kbd_SW_Hole:Stab_Hole_Choc_2u_Top
- added Ref**: Val**, kbd_Hole:m2_Screw_Hole, F.Cu at (181.0, 23.8)
- added Ref**: Val**, kbd_Hole:m2_Screw_Hole, F.Cu at (88.1, 23.8)
- added SW**: SW_PUSH, kbd_SW_Hole:Stab_Hole_Choc_2u_Top, F.Cu at (140.5, 133.3)
- added SW**: SW_PUSH, kbd_SW_Hole:Stab_Hole_Choc_2u_Top, F.Cu at (42.9, 114.3)
- SW10, SW15, SW20, SW5: footprint kbd_SW_Hole:SW_Hole_1u -> kbd_SW_Hole:SW_Hole_1.25u
- SW2: footprint kbd_SW_Hole:SW_Hole_1u -> kbd_SW_Hole:SW_Hole_1.5u
- SW3: footprint kbd_SW_Hole:SW_Hole_1u -> kbd_SW_Hole:SW_Hole_1.75u
- moved Ref** 47.6 mm to (133.3, 47.6)
Other:
- board size 164.3 x 102.4 mm -> 164.3 x 126.2 mm
