File: RKD_01/RKD01_Bottom_L/RKD01_Bottom_L.kicad_sch (KiCad schematic)
At the start: 72 parts, among them J1 TRRS, SW1 SW_Push, SW10 SW_Push, SW11 SW_Push, SW12 SW_Push, SW13 SW_Push, SW14 SW_Push, SW15 SW_Push, SW16 SW_Push, SW17 SW_Push, SW18 SW_Push, SW19 SW_Push, SW2 SW_Push, SW20 SW_Push, SW21 SW_Push, SW22 SW_Push, SW23 SW_Push, SW24 SW_Push, SW25 SW_Push, SW26 SW_Push, SW27 SW_Push, SW28 SW_Push, SW29 SW_Push, SW3 SW_Push, SW30 SW_Push, SW31 SW_Push, SW32 SW_Push, SW33 SW_Push, SW34 RotaryEncoder_Switch, SW35 SW_Push, SW4 SW_Push, SW5 SW_Push, SW6 SW_Push, SW7 SW_Push, SW8 SW_Push, SW9 SW_Push, U1 ProMicro

Commit message: 不要な情報を削除
Parts:
- removed D1, D10, D11, D12, D13, D14, D15, D16, D17, D18, D19, D2, D20, D21, D22, D23, D24, D25, D26, D27, D28, D29, D3, D30, D31, D32, D33, D34, D4, D5, D6, D7, D8, D9: D, kbd_Parts:Diode_SMD, symbol Device:D
- removed J1: TRRS, BrownSugar_KBD:TRRS_PJ-320A, symbol BrownSugar_KBD:TRRS
- removed OL1: OLED, BrownSugar_KBD:OLED_center_module, symbol BrownSugar_KBD:OLED
- removed SW1, SW10, SW11, SW12, SW13, SW14, SW15, SW16, SW17, SW18, SW19, SW2, SW20, SW21, SW22, SW23, SW24, SW26, SW27, SW28, SW29, SW3, SW30, SW31, SW32, SW33, SW5, SW6, SW7, SW8, SW9: SW_Push, kbd_SW:Choc_Hotswap_1u, symbol Switch:SW_Push
- removed SW25, SW4: SW_Push, kbd_SW:Choc_Hotswap_2u_Stab, symbol Switch:SW_Push
- removed SW34: RotaryEncoder_Switch, BrownSugar_KBD:RotaryEncoder_EC11-Switch, symbol Device:RotaryEncoder_Switch
- removed SW35: SW_Push, kbd_Parts:ResetSW, symbol Switch:SW_Push
- removed U1: ProMicro, BrownSugar_KBD:ProMicro_r, symbol BrownSugar_KBD:ProMicro
Connections:
- no-connect marks 2 -> 0
