File: RKD_01/RKD01_Right_Greed01/RKD01_Top_R/RKD01_Top_R.kicad_pcb (KiCad board)
At the start: 2 copper layers, 197.6 x 126.2 mm, 54 parts, among them M1 Mark, M2 Mark, M3 Mark, M4 Mark, M5 Mark, M6 Mark, M7 Mark, M8 Mark, SW36 SW_Push, SW37 SW_Push, SW38 SW_Push, SW39 SW_Push, SW40 SW_Push, SW41 SW_Push, SW42 SW_Push, SW43 SW_Push, SW44 SW_Push, SW45 SW_Push, SW46 SW_Push, SW47 SW_Push, SW48 SW_Push, SW49 SW_Push, SW50 SW_Push, SW51 SW_Push, SW52 SW_Push, SW53 SW_Push, SW54 SW_Push, SW55 SW_Push, SW56 SW_Push, SW57 SW_Push, SW58 SW_Push, SW59 SW_Push, SW60 SW_Push, SW61 SW_Push, SW62 SW_Push, SW63 SW_Push, SW64 SW_Push, SW65 SW_Push, SW66 SW_Push, SW67 SW_Push, SW68 SW_Push, SW69 SW_Push, SW70 SW_Push, SW71 SW_Push, SW72 SW_Push, SW73 SW_Push, SW74 SW_Push, SW75 SW_Push, SW76 SW_Push

Commit message: az1uball用の穴サイズ変更
Parts:
- Trackball1: footprint kbd_SW_Hole:SW_Hole_1u -> kbd_SW_Hole:az_hole
Changed lines of the file:
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@@
 		)
 	)
-	(footprint "kbd_SW_Hole:SW_Hole_1u"
+	(footprint "kbd_SW_Hole:az_hole"
 		(layer "F.Cu")
 		(at 28.575 114.3)
@@
 			)
 		)
-		(property "Footprint" "kbd_SW_Hole:SW_Hole_1u"
+		(property "Footprint" "kbd_SW_Hole:az_hole"
 			(at 0 0 0)
 			(layer "F.Fab")
@@
 		(attr through_hole)
 		(fp_line
-			(start -7.05 -7.05)
-			(end 7.05 -7.05)
+			(start -8.05 -8.05)
+			(end 8.05 -8.05)
 			(stroke
 				(width 0.15)
@@
 		)
 		(fp_line
-			(start -7.05 7.05)
-			(end -7.05 -7.05)
+			(start -8.05 8.05)
+			(end -8.05 -8.05)
 			(stroke
 				(width 0.15)
@@
 		)
 		(fp_line
-			(start 7.05 -7.05)
-			(end 7.05 7.05)
+			(start 8.05 -8.05)
+			(end 8.05 8.05)
 			(stroke
 				(width 0.15)
@@
 		)
 		(fp_line
-			(start 7.05 7.05)
-			(end -7.05 7.05)
+			(start 8.05 8.05)
+			(end -8.05 8.05)
 			(stroke
 				(width 0.15)

Commit message: 寸法を見直し
Parts:
- removed SW** (x2): SW_PUSH, kbd_SW_Hole:Stab_Hole_Choc_2u_Top
- removed the Trackball1 at (28.6, 114.3)
- removed the Trackball1 at (33.3, 133.3)
- added SW37: SW_Push, kbd_SW_Hole:SW_Hole_1u, F.Cu at (45.2, 76.2)
- added SW40: SW_Push, kbd_SW_Hole:SW_Hole_1u, F.Cu at (40.5, 133.3)
- added SW66: SW_PUSH, kbd_SW_Hole:Stab_Hole_Choc_2u_Top, F.Cu at (195.3, 95.2)
- added SW66: SW_PUSH, kbd_SW_Hole:Stab_Hole_Choc_2u_Top, F.Cu at (197.6, 57.1)
- SW41: renamed from SW39; footprint kbd_SW_Hole:SW_Hole_1.5u -> kbd_SW_Hole:SW_Hole_1u
- SW45: renamed from SW43; footprint kbd_SW_Hole:SW_Hole_1u -> kbd_SW_Hole:SW_Hole_1.5u
- Trackball1: footprint kbd_SW_Hole:SW_Hole_1u -> kbd_SW_Hole:az_hole
- moved SW41 76.2 mm to (54.8, 57.1)
- moved M6 64.3 mm to (154.8, 104.8)
- moved M4 54.8 mm to (154.8, 47.6)
- moved M5 50.0 mm to (92.9, 85.7)
- moved M3 40.5 mm to (31.0, 47.6)
- moved Trackball1 38.2 mm to (35.7, 114.3), turned to -90 degrees
- moved SW42 25.3 mm to (64.3, 76.2)
- moved SW43 22.5 mm to (69.1, 95.2)
- moved SW44 22.5 mm to (73.8, 114.3)
- moved SW45 19.2 mm to (64.3, 133.3)
- moved M8 9.53 mm to (219.1, 140.5)
- moved M2 9.52 mm to (219.1, 23.8)
- moved SW50 7.14 mm to (95.3, 133.3)
- moved SW55 7.14 mm to (123.8, 133.3)
- moved SW64 7.14 mm to (147.6, 133.3)
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- renumbered SW37 to SW38, SW38 to SW39, SW40 to SW42, SW41 to SW43, SW42 to SW44, SW44 to SW46, SW45 to SW47, SW46 to SW48, SW47 to SW49, SW48 to SW50, SW49 to SW51, SW50 to SW52, SW51 to SW53, SW52 to SW54, SW53 to SW55, SW54 to SW56, SW55 to SW57, SW56 to SW58, SW57 to SW59, SW58 to SW60, SW59 to SW61, SW60 to SW62, SW61 to SW63, SW62 to SW64, SW63 to SW65, SW64 to SW66, SW65 to SW67, SW66 to SW68, SW67 to SW69, SW68 to SW70, SW69 to SW71, SW70 to SW72, SW71 to SW73, SW72 to SW74, SW73 to SW75, SW74 to SW76, SW75 to SW77, SW76 to SW78
Other:
- board size 197.6 x 126.2 mm -> 202.4 x 126.2 mm
- board text added: "RKD01_Right_B v1.0"

Commit message: az用holeを自作分に変更
Parts:
- Trackball1: footprint kbd_SW_Hole:az_hole -> Rikkodo_FootPrint:rkd_az_hole
Changed lines of the file:
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@@
 		)
 	)
-	(footprint "kbd_SW_Hole:az_hole"
+	(footprint "Rikkodo_FootPrint:rkd_az_hole"
 		(layer "F.Cu")
 		(at 35.7188 114.3 -90)
@@
 			)
 		)
-		(property "Footprint" "kbd_SW_Hole:az_hole"
+		(property "Footprint" "Rikkodo_FootPrint:rkd_az_hole"
 			(at 0 0 -90)
 			(layer "F.Fab")
