File: RKD_01/RKD01_Right_Greed01/RKD01_Assemble_R/RKD01_Assemble_R.kicad_sch (KiCad schematic)
At the start: 101 parts, among them J2 TRRS, M1 Mark, M10 Mark, M2 Mark, M3 Mark, M4 Mark, M5 Mark, M6 Mark, M7 Mark, M8 Mark, M9 Mark, SW36 SW_Push, SW37 SW_Push, SW38 SW_Push, SW39 SW_Push, SW40 SW_Push, SW41 SW_Push, SW42 SW_Push, SW43 SW_Push, SW44 SW_Push, SW45 SW_Push, SW46 SW_Push, SW47 SW_Push, SW48 SW_Push, SW49 SW_Push, SW50 SW_Push, SW51 SW_Push, SW52 SW_Push, SW53 SW_Push, SW54 SW_Push, SW55 SW_Push, SW56 SW_Push, SW57 SW_Push, SW58 SW_Push, SW59 SW_Push, SW60 SW_Push, SW61 SW_Push, SW62 SW_Push, SW63 SW_Push, SW64 SW_Push, SW65 SW_Push, SW66 SW_Push, SW67 SW_Push, SW68 SW_Push, SW69 SW_Push, SW70 SW_Push, SW71 SW_Push, SW72 SW_Push, SW73 SW_Push, SW74 SW_Push, SW75 SW_Push, SW76 SW_Push, SW77 SW_Push, SW78 SW_Push, SW79 SW_Push, U2 ProMicro

Commit message: デザイン見直し
Parts:
- removed M5, M6, M7, M8: Mark, kbd_Hole:m2_Spacer_Hole_hex, symbol BrownSugar_KBD:Mark
- removed OL2: OLED, BrownSugar_KBD:OLED_center_module, symbol BrownSugar_KBD:OLED
- removed SW79: SW_Push, kbd_Parts:ResetSW, symbol Switch:SW_Push
- renumbered M9 to M5, M10 to M6
Connections:
- net Reset: no longer names the net of U2.22 (RST)
- no-connect marks 2 -> 3
