File: RKD_01/RKD01_Common/RKD01_AzHoot/RKD01_AzHoot.kicad_sch (KiCad schematic)
At the start: 3 parts, among them M1 Mark, P1 pointing

Commit message: 足場をカットに更新
Parts:
- M1: footprint Rikkodo_FootPrint:rkd_Point_Hall -> Rikkodo_FootPrint:rkd_Point_Cut
Changed lines of the file:
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@@
 			)
 		)
-		(property "Footprint" "Rikkodo_FootPrint:rkd_Point_Hall"
+		(property "Footprint" "Rikkodo_FootPrint:rkd_Point_Cut"
 			(at 105.41 50.8 0)
 			(effects
