File: RKD_01/RKD01_Right/RKD01_Assemble_R_Ball/RKD01_Assemble_R_Ball.kicad_sch (KiCad schematic)
At the start: 95 parts, among them J2 TRRS, M1 Mark, M2 Mark, M3 Mark, M4 Mark, M5 Mark, M6 Mark, SW36 SW_Push, SW37 SW_Push, SW38 SW_Push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

Commit message: スイッチ番号の見直し
Parts:
- renumbered D36 to D51, D37 to D52, D38 to D53, D39 to D54, D40 to D55, D41 to D56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
