File: RKD_01/RKD01_Right/RKD01_Assemble_R/RKD01_Assemble_R.kicad_sch (KiCad schematic)
At the start: 98 parts, among them J2 TRRS, M1 Mark, M2 Mark, M3 Mark, M4 Mark, M5 Mark, M6 Mark, P1 pointing, SW51 SW_Push, SW52 SW_Push, SW53 SW_Push, SW54 SW_Push, SW55 SW_Push, SW56 SW_Push, SW57 SW_Push, SW58 SW_Push, SW59 SW_Push, SW60 SW_Push, SW61 SW_Push, SW62 SW_Push, SW63 SW_Push, SW64 SW_Push, SW65 SW_Push, SW66 SW_Push, SW67 SW_Push, SW68 SW_Push, SW69 SW_Push, SW70 SW_Push, SW71 SW_Push, SW72 SW_Push, SW73 SW_Push, SW74 SW_Push, SW75 SW_Push, SW76 SW_Push, SW77 SW_Push, SW78 SW_Push, SW79 SW_Push, SW80 SW_Push, SW81 SW_Push, SW82 SW_Push, SW83 SW_Push, SW84 SW_Push, SW85 SW_Push, SW86 SW_Push, SW87 SW_Push, SW88 SW_Push, SW89 SW_Push, SW90 SW_Push, SW91 SW_Push, SW92 SW_Push, SW94 SW_Push, SW95 SW_Push, U2 ProMicro

Commit message: v1v2に修正
Parts:
- SW51, SW52, SW53, SW54, SW55, SW56, SW57, SW58, SW59, SW60, SW61, SW62, SW63, SW64, SW65, SW66, SW67, SW68, SW69, SW70, SW71, SW72, SW73, SW74, SW75, SW76, SW77, SW78, SW79, SW80, SW81, SW82, SW83, SW84, SW85, SW86, SW87, SW89, SW90, SW92, SW94, SW95: footprint Rikkodo_FootPrint:rkd_Choc_v2_Hotswap_1u -> Rikkodo_FootPrint:rkd_Choc_v1v2_Hotswap_1u
- SW88, SW91: footprint Rikkodo_FootPrint:rkd_Choc_v2_Hotswap_2u -> Rikkodo_FootPrint:rkd_Choc_v1v2_Hotswap_2u
Changed lines of the file:
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@@
 			)
 		)
-		(property "Footprint" "Rikkodo_FootPrint:rkd_Choc_v2_Hotswap_1u"
+		(property "Footprint" "Rikkodo_FootPrint:rkd_Choc_v1v2_Hotswap_1u"
 			(at 254 198.12 0)
 			(effects
@@
 			)
 		)
-		(property "Footprint" "Rikkodo_FootPrint:rkd_Choc_v2_Hotswap_1u"
+		(property "Footprint" "Rikkodo_FootPrint:rkd_Choc_v1v2_Hotswap_1u"
 			(at 127 198.12 0)
 			(effects
@@
 			)
 		)
-		(property "Footprint" "Rikkodo_FootPrint:rkd_Choc_v2_Hotswap_1u"
+		(property "Footprint" "Rikkodo_FootPrint:rkd_Choc_v1v2_Hotswap_1u"
 			(at 76.2 223.52 0)
 			(effects
@@
 			)
 		)
-		(property "Footprint" "Rikkodo_FootPrint:rkd_Choc_v2_Hotswap_1u"
+		(property "Footprint" "Rikkodo_FootPrint:rkd_Choc_v1v2_Hotswap_1u"
 			(at 101.6 172.72 0)
 			(effects
@@
 			)
 		)
-		(property "Footprint" "Rikkodo_FootPrint:rkd_Choc_v2_Hotswap_1u"
+		(property "Footprint" "Rikkodo_FootPrint:rkd_Choc_v1v2_Hotswap_1u"
 			(at 101.6 147.32 0)
 			(effects
@@
 			)
 		)
-		(property "Footprint" "Rikkodo_FootPrint:rkd_Choc_v2_Hotswap_2u"
+		(property "Footprint" "Rikkodo_FootPrint:rkd_Choc_v1v2_Hotswap_2u"
 			(at 228.6 172.72 0)
 			(effects
@@
 			)
 		)
-		(property "Footprint" "Rikkodo_FootPrint:rkd_Choc_v2_Hotswap_1u"
+		(property "Footprint" "Rikkodo_FootPrint:rkd_Choc_v1v2_Hotswap_1u"
 			(at 203.2 147.32 0)
 			(effects
@@
 			)
 		)
-		(property "Footprint" "Rikkodo_FootPrint:rkd_Choc_v2_Hotswap_1u"
+		(property "Footprint" "Rikkodo_FootPrint:rkd_Choc_v1v2_Hotswap_1u"
 			(at 203.2 172.72 0)
 			(effects
@@
 			)
 		)
-		(property "Footprint" "Rikkodo_FootPrint:rkd_Choc_v2_Hotswap_1u"
+		(property "Footprint" "Rikkodo_FootPrint:rkd_Choc_v1v2_Hotswap_1u"
 			(at 177.8 172.72 0)
 			(effects
@@
 			)
 		)
-		(property "Footprint" "Rikkodo_FootPrint:rkd_Choc_v2_Hotswap_1u"
+		(property "Footprint" "Rikkodo_FootPrint:rkd_Choc_v1v2_Hotswap_1u"
 			(at 76.2 147.32 0)
 			(effects
@@
 			)
 		)
-		(property "Footprint" "Rikkodo_FootPrint:rkd_Choc_v2_Hotswap_1u"
+		(property "Footprint" "Rikkodo_FootPrint:rkd_Choc_v1v2_Hotswap_1u"
 			(at 50.8 198.12 0)
 			(effects
@@
 			)
 		)
-		(property "Footprint" "Rikkodo_FootPrint:rkd_Choc_v2_Hotswap_1u"
+		(property "Footprint" "Rikkodo_FootPrint:rkd_Choc_v1v2_Hotswap_1u"
 			(at 177.8 223.52 0)
 			(effects
@@
 			)
 		)
-		(property "Footprint" "Rikkodo_FootPrint:rkd_Choc_v2_Hotswap_1u"
+		(property "Footprint" "Rikkodo_FootPrint:rkd_Choc_v1v2_Hotswap_1u"
 			(at 177.8 198.12 0)
 			(effects
@@
 			)
 		)
-		(property "Footprint" "Rikkodo_FootPrint:rkd_Choc_v2_Hotswap_1u"
+		(property "Footprint" "Rikkodo_FootPrint:rkd_Choc_v1v2_Hotswap_1u"
 			(at 228.6 147.32 0)
 			(effects
@@
 			)
 		)
-		(property "Footprint" "Rikkodo_FootPrint:rkd_Choc_v2_Hotswap_1u"
+		(property "Footprint" "Rikkodo_FootPrint:rkd_Choc_v1v2_Hotswap_1u"
 			(at 127 147.32 0)
 			(effects
@@
 			)
 		)
-		(property "Footprint" "Rikkodo_FootPrint:rkd_Choc_v2_Hotswap_1u"
+		(property "Footprint" "Rikkodo_FootPrint:rkd_Choc_v1v2_Hotswap_1u"
 			(at 254 147.32 0)
 			(effects
@@
 			)
 		)
-		(property "Footprint" "Rikkodo_FootPrint:rkd_Choc_v2_Hotswap_1u"
+		(property "Footprint" "Rikkodo_FootPrint:rkd_Choc_v1v2_Hotswap_1u"
 			(at 177.8 121.92 0)
 			(effects
@@
 			)
 		)
-		(property "Footprint" "Rikkodo_FootPrint:rkd_Choc_v2_Hotswap_1u"
+		(property "Footprint" "Rikkodo_FootPrint:rkd_Choc_v1v2_Hotswap_1u"
 			(at 50.8 223.52 0)
 			(effects
@@
 			)
 		)
-		(property "Footprint" "Rikkodo_FootPrint:rkd_Choc_v2_Hotswap_1u"
+		(property "Footprint" "Rikkodo_FootPrint:rkd_Choc_v1v2_Hotswap_1u"
 			(at 177.8 147.32 0)
 			(effects
@@
 			)
 		)
-		(property "Footprint" "Rikkodo_FootPrint:rkd_Choc_v2_Hotswap_1u"
+		(property "Footprint" "Rikkodo_FootPrint:rkd_Choc_v1v2_Hotswap_1u"
 			(at 101.6 198.12 0)
 			(effects
@@
 			)
 		)
-		(property "Footprint" "Rikkodo_FootPrint:rkd_Choc_v2_Hotswap_1u"
+		(property "Footprint" "Rikkodo_FootPrint:rkd_Choc_v1v2_Hotswap_1u"
 			(at 152.4 147.32 0)
 			(effects
@@
 			)
 		)
-		(property "Footprint" "Rikkodo_FootPrint:rkd_Choc_v2_Hotswap_1u"
+		(property "Footprint" "Rikkodo_FootPrint:rkd_Choc_v1v2_Hotswap_1u"
 			(at 76.2 198.12 0)
 			(effects
@@
 			)
 		)
-		(property "Footprint" "Rikkodo_FootPrint:rkd_Choc_v2_Hotswap_1u"
+		(property "Footprint" "Rikkodo_FootPrint:rkd_Choc_v1v2_Hotswap_1u"
 			(at 228.6 198.12 0)
 			(effects
@@
 			)
 		)
-		(property "Footprint" "Rikkodo_FootPrint:rkd_Choc_v2_Hotswap_1u"
+		(property "Footprint" "Rikkodo_FootPrint:rkd_Choc_v1v2_Hotswap_1u"
 			(at 203.2 223.52 0)
 			(effects
@@
 			)
 		)
-		(property "Footprint" "Rikkodo_FootPrint:rkd_Choc_v2_Hotswap_1u"
+		(property "Footprint" "Rikkodo_FootPrint:rkd_Choc_v1v2_Hotswap_1u"
 			(at 127 223.52 0)
 			(effects
@@
 			)
 		)
-		(property "Footprint" "Rikkodo_FootPrint:rkd_Choc_v2_Hotswap_1u"
+		(property "Footprint" "Rikkodo_FootPrint:rkd_Choc_v1v2_Hotswap_1u"
 			(at 50.8 147.32 0)
 			(effects
@@
 			)
 		)
-		(property "Footprint" "Rikkodo_FootPrint:rkd_Choc_v2_Hotswap_1u"
+		(property "Footprint" "Rikkodo_FootPrint:rkd_Choc_v1v2_Hotswap_1u"
 			(at 76.2 172.72 0)
 			(effects
@@
 			)
 		)
-		(property "Footprint" "Rikkodo_FootPrint:rkd_Choc_v2_Hotswap_1u"
+		(property "Footprint" "Rikkodo_FootPrint:rkd_Choc_v1v2_Hotswap_1u"
 			(at 101.6 223.52 0)
 			(effects
@@
 			)
 		)
-		(property "Footprint" "Rikkodo_FootPrint:rkd_Choc_v2_Hotswap_1u"
+		(property "Footprint" "Rikkodo_FootPrint:rkd_Choc_v1v2_Hotswap_1u"
 			(at 203.2 121.92 0)
 			(effects
@@
 			)
 		)
-		(property "Footprint" "Rikkodo_FootPrint:rkd_Choc_v2_Hotswap_1u"
+		(property "Footprint" "Rikkodo_FootPrint:rkd_Choc_v1v2_Hotswap_1u"
 			(at 254 223.52 0)
 			(effects
@@
 			)
 		)
-		(property "Footprint" "Rikkodo_FootPrint:rkd_Choc_v2_Hotswap_1u"
+		(property "Footprint" "Rikkodo_FootPrint:rkd_Choc_v1v2_Hotswap_1u"
 			(at 203.2 198.12 0)
 			(effects
@@
 			)
 		)
-		(property "Footprint" "Rikkodo_FootPrint:rkd_Choc_v2_Hotswap_1u"
+		(property "Footprint" "Rikkodo_FootPrint:rkd_Choc_v1v2_Hotswap_1u"
 			(at 228.6 223.52 0)
 			(effects
@@
 			)
 		)
-		(property "Footprint" "Rikkodo_FootPrint:rkd_Choc_v2_Hotswap_1u"
+		(property "Footprint" "Rikkodo_FootPrint:rkd_Choc_v1v2_Hotswap_1u"
 			(at 152.4 198.12 0)
 			(effects
@@
 			)
 		)
-		(property "Footprint" "Rikkodo_FootPrint:rkd_Choc_v2_Hotswap_2u"
+		(property "Footprint" "Rikkodo_FootPrint:rkd_Choc_v1v2_Hotswap_2u"
 			(at 254 121.92 0)
 			(effects
@@
 			)
 		)
-		(property "Footprint" "Rikkodo_FootPrint:rkd_Choc_v2_Hotswap_1u"
+		(property "Footprint" "Rikkodo_FootPrint:rkd_Choc_v1v2_Hotswap_1u"
 			(at 152.4 121.92 0)
 			(effects
@@
 			)
 		)
-		(property "Footprint" "Rikkodo_FootPrint:rkd_Choc_v2_Hotswap_1u"
+		(property "Footprint" "Rikkodo_FootPrint:rkd_Choc_v1v2_Hotswap_1u"
 			(at 101.6 121.92 0)
 			(effects
@@
 			)
 		)
-		(property "Footprint" "Rikkodo_FootPrint:rkd_Choc_v2_Hotswap_1u"
+		(property "Footprint" "Rikkodo_FootPrint:rkd_Choc_v1v2_Hotswap_1u"
 			(at 50.8 121.92 0)
 			(effects
@@
 			)
 		)
-		(property "Footprint" "Rikkodo_FootPrint:rkd_Choc_v2_Hotswap_1u"
+		(property "Footprint" "Rikkodo_FootPrint:rkd_Choc_v1v2_Hotswap_1u"
 			(at 127 172.72 0)
 			(effects
@@
 			)
 		)
-		(property "Footprint" "Rikkodo_FootPrint:rkd_Choc_v2_Hotswap_1u"
+		(property "Footprint" "Rikkodo_FootPrint:rkd_Choc_v1v2_Hotswap_1u"
 			(at 228.6 121.92 0)
 			(effects
@@
 			)
 		)
-		(property "Footprint" "Rikkodo_FootPrint:rkd_Choc_v2_Hotswap_1u"
+		(property "Footprint" "Rikkodo_FootPrint:rkd_Choc_v1v2_Hotswap_1u"
 			(at 127 121.92 0)
 			(effects
@@
 			)
 		)
-		(property "Footprint" "Rikkodo_FootPrint:rkd_Choc_v2_Hotswap_1u"
+		(property "Footprint" "Rikkodo_FootPrint:rkd_Choc_v1v2_Hotswap_1u"
 			(at 152.4 172.72 0)
 			(effects
@@
 			)
 		)
-		(property "Footprint" "Rikkodo_FootPrint:rkd_Choc_v2_Hotswap_1u"
+		(property "Footprint" "Rikkodo_FootPrint:rkd_Choc_v1v2_Hotswap_1u"
 			(at 152.4 223.52 0)
 			(effects
@@
 			)
 		)
-		(property "Footprint" "Rikkodo_FootPrint:rkd_Choc_v2_Hotswap_1u"
+		(property "Footprint" "Rikkodo_FootPrint:rkd_Choc_v1v2_Hotswap_1u"
 			(at 50.8 172.72 0)
 			(effects
@@
 			)
 		)
-		(property "Footprint" "Rikkodo_FootPrint:rkd_Choc_v2_Hotswap_1u"
+		(property "Footprint" "Rikkodo_FootPrint:rkd_Choc_v1v2_Hotswap_1u"
 			(at 76.2 121.92 0)
 			(effects
