File: RKD_03/RKD03_Assemble/RKD03_Assemble.kicad_sch (KiCad schematic)
At the start: 29 parts, among them J1 GROVE-CONNECTOR-DIP_4P-2.0_, SW1 SW_Push, SW10 SW_Push, SW2 SW_Push, SW3 SW_Push, SW4 SW_Push, SW5 SW_Push, SW6 SW_Push, SW7 SW_Push, SW8 SW_Push, SW9 SW_Push, U1 Pico

Commit message: RKD03修正
Parts:
- added M1: Mark, Rikkodo_FootPrint:rkd_Guard_Screw_Hall, symbol BrownSugar_KBD:Mark
- SW1, SW3, SW5, SW7, SW9: footprint Rikkodo_FootPrint:rkd_CherryChoc_v1v2_Hotswap_1u -> Rikkodo_FootPrint:rkd_Choc_v1v2_Hotswap_2u_Gat
- SW10, SW2, SW4, SW6, SW8: footprint Rikkodo_FootPrint:rkd_CherryChoc_v1v2_Hotswap_1u -> Rikkodo_FootPrint:rkd_Choc_v1v2_Hotswap_1u
- U1: footprint RPi_Pico:RPi_Pico_SMD_TH -> Rikkodo_FootPrint:rkd_RPi_Pico_TH
Connections:
- net 3v3: now also J1.2; no longer J1.3
- net GND: now also J1.1; no longer J1.4, U1.23 (GND), U1.28 (GND), U1.38 (GND)
- net SCL: now also J1.4; no longer J1.2
- net SDA: now also J1.3; no longer J1.1
- no-connect marks 25 -> 27
Changed lines of the file:
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@@
 	)
 	(junction
-		(at 101.6 57.15)
-		(diameter 0)
-		(color 0 0 0 0)
-	)
-	(junction
 		(at 60.96 241.3)
 		(diameter 0)
@@
 	)
 	(junction
-		(at 101.6 69.85)
-		(diameter 0)
-		(color 0 0 0 0)
-	)
-	(junction
 		(at 185.42 63.5)
 		(diameter 0)
@@
 	)
 	(no_connect
+		(at 83.82 57.15)
+	)
+	(no_connect
 		(at 83.82 67.31)
 	)
+	(no_connect
+		(at 83.82 69.85)
+	)
 	(wire
 		(pts
@@
 	(wire
 		(pts
-			(xy 83.82 57.15) (xy 101.6 57.15)
-		)
-		(stroke
-			(width 0)
-			(type default)
-		)
-	)
-	(wire
-		(pts
 			(xy 25.4 69.85) (xy 48.26 69.85)
 		)
@@
 	(wire
 		(pts
-			(xy 105.41 128.27) (xy 123.19 128.27)
-		)
-		(stroke
-			(width 0)
-			(type default)
-		)
-	)
-	(wire
-		(pts
 			(xy 76.2 233.68) (xy 76.2 259.08)
 		)
@@
 	(wire
 		(pts
-			(xy 101.6 69.85) (xy 101.6 88.9)
+			(xy 114.3 123.19) (xy 114.3 139.7)
 		)
 		(stroke
@@
 	(wire
 		(pts
-			(xy 66.04 266.7) (xy 91.44 266.7)
+			(xy 123.19 123.19) (xy 114.3 123.19)
 		)
 		(stroke
@@
 	(wire
 		(pts
-			(xy 38.1 241.3) (xy 60.96 241.3)
+			(xy 66.04 266.7) (xy 91.44 266.7)
 		)
 		(stroke
@@
 	(wire
 		(pts
-			(xy 83.82 69.85) (xy 101.6 69.85)
+			(xy 38.1 241.3) (xy 60.96 241.3)
 		)
 		(stroke
@@
 	(wire
 		(pts
-			(xy 101.6 31.75) (xy 101.6 57.15)
-		)
-		(stroke
-			(width 0)
-			(type default)
-		)
-	)
-	(wire
-		(pts
-			(xy 83.82 31.75) (xy 101.6 31.75)
-		)
-		(stroke
-			(width 0)
-			(type default)
-		)
-	)
-	(wire
-		(pts
 			(xy 25.4 44.45) (xy 25.4 57.15)
 		)
@@
 	(wire
 		(pts
-			(xy 101.6 57.15) (xy 101.6 69.85)
-		)
-		(stroke
-			(width 0)
-			(type default)
-		)
-	)
-	(wire
-		(pts
 			(xy 25.4 69.85) (xy 25.4 88.9)
 		)
@@
 		)
 	)
-	(global_label "SDA"
+	(global_label "Col4"
 		(shape input)
-		(at 123.19 123.19 180)
+		(at 152.4 195.58 180)
 		(fields_autoplaced yes)
 		(effects
@@
 		)
 		(property "Intersheetrefs" "${INTERSHEET_REFS}"
-			(at 116.6367 123.19 0)
+			(at 145.1211 195.58 0)
 			(effects
 				(font
@@
 		)
 	)
-	(global_label "Col4"
+	(global_label "SDA"
 		(shape input)
-		(at 152.4 195.58 180)
+		(at 123.19 128.27 180)
 		(fields_autoplaced yes)
 		(effects
@@
 		)
 		(property "Intersheetrefs" "${INTERSHEET_REFS}"
-			(at 145.1211 195.58 0)
+			(at 116.6367 128.27 0)
 			(effects
 				(font
@@
 		)
 	)
-	(global_label "SDA"
+	(global_label "SCL"
 		(shape input)
-		(at 144.78 58.42 180)
+		(at 123.19 130.81 180)
 		(fields_autoplaced yes)
 		(effects
@@
 		)
 		(property "Intersheetrefs" "${INTERSHEET_REFS}"
-			(at 138.2267 58.42 0)
+			(at 116.6972 130.81 0)
 			(effects
 				(font
@@
 		)
 	)
-	(global_label "SCL"
+	(global_label "SDA"
 		(shape input)
-		(at 123.19 125.73 180)
+		(at 144.78 58.42 180)
 		(fields_autoplaced yes)
 		(effects
@@
 		)
 		(property "Intersheetrefs" "${INTERSHEET_REFS}"
-			(at 116.6972 125.73 0)
+			(at 138.2267 58.42 0)
 			(effects
 				(font
@@
 	(global_label "3v3"
 		(shape input)
-		(at 105.41 128.27 180)
+		(at 123.19 125.73 180)
 		(fields_autoplaced yes)
 		(effects
@@
 		)
 		(property "Intersheetrefs" "${INTERSHEET_REFS}"
-			(at 99.0382 128.27 0)
+			(at 116.8182 125.73 0)
 			(effects
 				(font
@@
 			)
 		)
-		(property "Footprint" "Rikkodo_FootPrint:rkd_CherryChoc_v1v2_Hotswap_1u"
+		(property "Footprint" "Rikkodo_FootPrint:rkd_Choc_v1v2_Hotswap_2u_Gat"
 			(at 81.28 228.6 0)
 			(effects
@@
 			)
 		)
-		(property "Footprint" "Rikkodo_FootPrint:rkd_CherryChoc_v1v2_Hotswap_1u"
+		(property "Footprint" "Rikkodo_FootPrint:rkd_Choc_v1v2_Hotswap_2u_Gat"
 			(at 157.48 228.6 0)
 			(effects
@@
 			)
 		)
-		(property "Footprint" "Rikkodo_FootPrint:rkd_CherryChoc_v1v2_Hotswap_1u"
+		(property "Footprint" "Rikkodo_FootPrint:rkd_Choc_v1v2_Hotswap_1u"
 			(at 86.36 254 0)
 			(effects
@@
 			)
 		)
-		(property "Footprint" "Rikkodo_FootPrint:rkd_CherryChoc_v1v2_Hotswap_1u"
+		(property "Footprint" "Rikkodo_FootPrint:rkd_Choc_v1v2_Hotswap_1u"
 			(at 162.56 254 0)
 			(effects
@@
 	)
 	(symbol
-		(lib_id "power:GND")
-		(at 101.6 88.9 0)
-		(unit 1)
-		(exclude_from_sim no)
-		(in_bom yes)
-		(on_board yes)
-		(dnp no)
-		(fields_autoplaced yes)
-		(property "Reference" "#PWR02"
-			(at 101.6 95.25 0)
-			(effects
-				(font
-					(size 1.27 1.27)
-				)
-				(hide yes)
-			)
-		)
-		(property "Value" "GND"
-			(at 101.6 93.98 0)
-			(effects
-				(font
-					(size 1.27 1.27)
-				)
-			)
-		)
-		(property "Footprint" ""
-			(at 101.6 88.9 0)
-			(effects
-				(font
-					(size 1.27 1.27)
-				)
-				(hide yes)
-			)
-		)
-		(property "Datasheet" ""
-			(at 101.6 88.9 0)
-			(effects
-				(font
-					(size 1.27 1.27)
-				)
-				(hide yes)
-			)
-		)
-		(property "Description" "Power symbol creates a global label with name \"GND\" , ground"
-			(at 101.6 88.9 0)
-			(effects
-				(font
-					(size 1.27 1.27)
-				)
-				(hide yes)
-			)
-		)
-		(pin "1"
-		)
-		(instances
-			(project ""
-				(path "/32b3db6f-ec5a-43c8-b598-c76dc9760296"
-					(reference "#PWR02")
-					(unit 1)
-				)
-			)
-		)
-	)
-	(symbol
 		(lib_id "RPi_Pico:Pico")
 		(at 66.04 50.8 0)
@@
 			)
 		)
-		(property "Footprint" "RPi_Pico:RPi_Pico_SMD_TH"
+		(property "Footprint" "Rikkodo_FootPrint:rkd_RPi_Pico_TH"
 			(at 66.04 50.8 90)
 			(effects
@@
 			)
 		)
-		(property "Footprint" "Rikkodo_FootPrint:rkd_CherryChoc_v1v2_Hotswap_1u"
+		(property "Footprint" "Rikkodo_FootPrint:rkd_Choc_v1v2_Hotswap_2u_Gat"
 			(at 106.68 228.6 0)
 			(effects
@@
 			)
 		)
-		(property "Footprint" "Rikkodo_FootPrint:rkd_CherryChoc_v1v2_Hotswap_1u"
+		(property "Footprint" "Rikkodo_FootPrint:rkd_Choc_v1v2_Hotswap_2u_Gat"
 			(at 132.08 228.6 0)
 			(effects
@@
 			)
 		)
-		(property "Footprint" "Rikkodo_FootPrint:rkd_CherryChoc_v1v2_Hotswap_1u"
+		(property "Footprint" "Rikkodo_FootPrint:rkd_Choc_v1v2_Hotswap_1u"
 			(at 137.16 254 0)
 			(effects
@@
 	(symbol
 		(lib_id "power:GND")
-		(at 123.19 130.81 0)
+		(at 114.3 139.7 0)
 		(unit 1)
 		(exclude_from_sim no)
@@
 		(fields_autoplaced yes)
 		(property "Reference" "#PWR014"
-			(at 123.19 137.16 0)
+			(at 114.3 146.05 0)
 			(effects
 				(font
@@
 		)
 		(property "Value" "GND"
-			(at 123.19 135.89 0)
+			(at 114.3 144.78 0)
 			(effects
 				(font
@@
 		)
 		(property "Footprint" ""
-			(at 123.19 130.81 0)
+			(at 114.3 139.7 0)
 			(effects
 				(font
@@
 		)
 		(property "Datasheet" ""
-			(at 123.19 130.81 0)
+			(at 114.3 139.7 0)
 			(effects
 				(font
@@
 		)
 		(property "Description" "Power symbol creates a global label with name \"GND\" , ground"
-			(at 123.19 130.81 0)
+			(at 114.3 139.7 0)
 			(effects
 				(font
@@
 			)
 		)
-		(property "Footprint" "Rikkodo_FootPrint:rkd_CherryChoc_v1v2_Hotswap_1u"
+		(property "Footprint" "Rikkodo_FootPrint:rkd_Choc_v1v2_Hotswap_1u"
 			(at 111.76 254 0)
 			(effects
@@
 			)
 		)
-		(property "Footprint" "Rikkodo_FootPrint:rkd_CherryChoc_v1v2_Hotswap_1u"
+		(property "Footprint" "Rikkodo_FootPrint:rkd_Choc_v1v2_Hotswap_1u"
 			(at 60.96 254 0)
 			(effects
@@
 			)
 		)
-		(property "Footprint" "Rikkodo_FootPrint:rkd_CherryChoc_v1v2_Hotswap_1u"
+		(property "Footprint" "Rikkodo_FootPrint:rkd_Choc_v1v2_Hotswap_2u_Gat"
 			(at 55.88 228.6 0)
 			(effects
@@
 					(unit 1)
 				)
+			)
+		)
+	)
+	(symbol
+		(lib_id "BrownSugar_KBD:Mark")
+		(at 231.14 124.46 0)
+		(unit 1)
+		(exclude_from_sim no)
+		(in_bom yes)
+		(on_board yes)
+		(dnp no)
+		(fields_autoplaced yes)
+		(property "Reference" "M1"
+			(at 233.68 123.1899 0)
+			(effects
+				(font
+					(size 1.27 1.27)
+				)
+				(justify left)
+			)
+		)
+		(property "Value" "Mark"
+			(at 233.68 125.7299 0)
+			(effects
+				(font
+					(size 1.27 1.27)
+				)
+				(justify left)
+			)
+		)
+		(property "Footprint" "Rikkodo_FootPrint:rkd_Guard_Screw_Hall"
+			(at 231.14 124.46 0)
+			(effects
+				(font
+					(size 1.27 1.27)
+				)
+			)
+		)
+		(property "Datasheet" ""
+			(at 231.14 124.46 0)
+			(effects
+				(font
+					(size 1.27 1.27)
+				)
+				(hide yes)
+			)
+		)
+		(property "Description" ""
+			(at 231.14 124.46 0)
+			(effects
+				(font
+					(size 1.27 1.27)
+				)
+				(hide yes)
+			)
+		)
+		(instances
+			(project ""
+				(path "/32b3db6f-ec5a-43c8-b598-c76dc9760296"
+					(reference "M1")
+					(unit 1)
+				)
