File: RKD_05/RKD05_Assemble/RKD05_Assemble.kicad_pcb (KiCad board)
At the start: 2 copper layers, 361.9 x 100 mm, 152 parts, among them J1 Conn_01x02_Socket, J3 Conn_01x24, M1 Mark, M2 Mark, M3 Mark, M4 Mark, M5 Mark, M6 Mark, M7 Mark, M8 Mark, SW1 SW_Push, SW10 SW_Push, SW11 SW_Push, SW12 SW_Push, SW13 SW_Push, SW14 SW_Push, SW15 SW_Push, SW16 SW_Push, SW17 SW_Push, SW18 SW_Push, SW19 SW_Push, SW2 SW_Push, SW20 SW_Push, SW21 SW_Push, SW22 SW_Push, SW23 SW_Push, SW24 SW_Push, SW25 SW_Push, SW26 SW_Push, SW27 SW_Push, SW28 SW_Push, SW29 SW_Push, SW3 SW_Push, SW30 SW_Push, SW4 SW_Push, SW40 RotaryEncoder_Switch, SW5 SW_Push, SW51 SW_Push, SW52 SW_Push, SW53 SW_Push, SW54 SW_Push, SW55 SW_Push, SW56 SW_Push, SW57 SW_Push, SW58 SW_Push, SW59 SW_Push, SW6 SW_Push, SW60 SW_Push, SW61 SW_Push, SW62 SW_Push, SW63 SW_Push, SW64 SW_Push, SW65 SW_Push, SW66 SW_Push, SW67 SW_Push, SW68 SW_Push, SW69 SW_Push, SW7 SW_Push, SW70 SW_Push, SW71 SW_Push, SW72 SW_Push, SW73 SW_Push, SW74 SW_Push, SW75 SW_Push, SW76 SW_Push, SW77 SW_Push, SW78 SW_Push, SW79 SW_Push, SW8 SW_Push, SW80 SW_Push, SW81 SW_Push, SW82 SW_Push, SW83 SW_Push, SW84 SW_Push, SW85 SW_Push, SW86 SW_Push, SW87 SW_Push, SW88 SW_Push, SW89 SW_Push, SW9 SW_Push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

Commit message: RKD05接続名変更
Connections:
- net 3v3 renamed PICOT:3v3
- net GND renamed PICOT:GND
- net RE1_A renamed PICOT:RE_A
- net RE1_B renamed PICOT:RE_B
- net VCC renamed PICOT:VCC
Changed lines of the file:
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@@
 	(net 69 "Net-(D90-A)")
 	(net 70 "GP19:SCL")
-	(net 71 "VCC")
-	(net 72 "GND")
-	(net 73 "RE1_A")
-	(net 74 "RE1_B")
+	(net 71 "PICOT:RE_B")
+	(net 72 "PICOT:RE_A")
+	(net 73 "PICOT:GND")
+	(net 74 "PICOT:3v3")
 	(net 75 "Net-(D88-A)")
 	(net 76 "GP18:SDA")
-	(net 77 "3v3")
+	(net 77 "PICOT:VCC")
 	(net 78 "unconnected-(SW40-PadS2)")
 	(net 79 "unconnected-(SW40-PadS1)")
@@
 			)
 			(remove_unused_layers no)
-			(net 77 "3v3")
+			(net 74 "PICOT:3v3")
 			(pinfunction "VCC")
 			(pintype "power_in")
@@
 			)
 			(remove_unused_layers no)
-			(net 72 "GND")
+			(net 73 "PICOT:GND")
 			(pinfunction "GND")
 			(pintype "power_in")
@@
 			)
 			(remove_unused_layers no)
-			(net 73 "RE1_A")
+			(net 72 "PICOT:RE_A")
 			(pinfunction "A")
 			(pintype "passive")
@@
 			)
 			(remove_unused_layers no)
-			(net 74 "RE1_B")
+			(net 71 "PICOT:RE_B")
 			(pinfunction "B")
 			(pintype "passive")
@@
 			)
 			(remove_unused_layers no)
-			(net 72 "GND")
+			(net 73 "PICOT:GND")
 			(pinfunction "C")
 			(pintype "passive")
@@
 			(size 0.3 1.3)
 			(layers "B.Cu" "B.Paste" "B.Mask")
-			(net 77 "3v3")
+			(net 74 "PICOT:3v3")
 			(pinfunction "Pin_22")
 			(pintype "passive")
@@
 			(size 0.3 1.3)
 			(layers "B.Cu" "B.Paste" "B.Mask")
-			(net 71 "VCC")
+			(net 77 "PICOT:VCC")
 			(pinfunction "Pin_23")
 			(pintype "passive")
@@
 			(size 0.3 1.3)
 			(layers "B.Cu" "B.Paste" "B.Mask")
-			(net 72 "GND")
+			(net 73 "PICOT:GND")
 			(pinfunction "Pin_24")
 			(pintype "passive")
@@
 		(tags "Through hole angled pin header THT 1x02 2.54mm single row")
 		(property "Reference" "J1"
-			(at 5.565626 1.701565 0)
+			(at 4.762636 -1.190485 0)
 			(layer "B.SilkS")
 			(effects
@@
 			)
 			(remove_unused_layers no)
-			(net 74 "RE1_B")
+			(net 71 "PICOT:RE_B")
 			(pinfunction "Pin_1")
 			(pintype "passive")
@@
 			)
 			(remove_unused_layers no)
-			(net 73 "RE1_A")
+			(net 72 "PICOT:RE_A")
 			(pinfunction "Pin_2")
 			(pintype "passive")
@@
 	)
 	(gr_text "RE_B"
-		(at 162.520449 169.664205 0)
+		(at 162.520176 170.556888 0)
 		(layer "B.SilkS")
 		(effects
@@
 	)
 	(segment
+		(start 163.353125 167.878125)
+		(end 166.56875 171.09375)
+		(width 0.25)
+		(layer "F.Cu")
+		(net 71)
+	)
+	(segment
+		(start 157.1625 167.878125)
+		(end 163.353125 167.878125)
+		(width 0.25)
+		(layer "F.Cu")
+		(net 71)
+	)
+	(segment
+		(start 165.813125 165.338125)
+		(end 157.1625 165.338125)
+		(width 0.25)
+		(layer "F.Cu")
+		(net 72)
+	)
+	(segment
+		(start 171.56875 171.09375)
+		(end 165.813125 165.338125)
+		(width 0.25)
+		(layer "F.Cu")
+		(net 72)
+	)
+	(segment
 		(start 148.490754 141.010855)
 		(end 148.490754 112.45)
 		(width 0.5)
 		(layer "B.Cu")
-		(net 72)
+		(net 73)
 	)
 	(segment
@@
 		(width 0.5)
 		(layer "B.Cu")
-		(net 72)
+		(net 73)
 	)
 	(segment
@@
 		(width 0.5)
 		(layer "B.Cu")
-		(net 72)
+		(net 73)
 	)
 	(segment
@@
 		(width 0.5)
 		(layer "B.Cu")
-		(net 72)
+		(net 73)
 	)
 	(segment
@@
 		(width 0.5)
 		(layer "B.Cu")
-		(net 72)
+		(net 73)
 	)
 	(segment
@@
 		(width 0.5)
 		(layer "B.Cu")
-		(net 72)
+		(net 73)
 	)
 	(segment
@@
 		(width 0.5)
 		(layer "B.Cu")
-		(net 72)
+		(net 73)
 	)
 	(segment
-		(start 165.813125 165.338125)
-		(end 157.1625 165.338125)
-		(width 0.25)
-		(layer "F.Cu")
-		(net 73)
+		(start 149.423563 140.493868)
+		(end 149.423563 113.704783)
+		(width 0.5)
+		(layer "B.Cu")
+		(net 74)
 	)
 	(segment
-		(start 171.56875 171.09375)
-		(end 165.813125 165.338125)
-		(width 0.25)
-		(layer "F.Cu")
-		(net 73)
+		(start 164.430951 150.614189)
+		(end 167.95764 147.0875)
+		(width 0.5)
+		(layer "B.Cu")
+		(net 74)
 	)
 	(segment
-		(start 163.353125 167.878125)
-		(end 166.56875 171.09375)
-		(width 0.25)
-		(layer "F.Cu")
+		(start 149.423563 140.493868)
+		(end 159.543884 150.614189)
+		(width 0.5)
+		(layer "B.Cu")
 		(net 74)
 	)
 	(segment
-		(start 157.1625 167.878125)
-		(end 163.353125 167.878125)
+		(start 149.423563 113.704783)
+		(end 149.590754 113.537592)
+		(width 0.5)
+		(layer "B.Cu")
+		(net 74)
+	)
+	(segment
+		(start 149.590754 112.45)
+		(end 149.590754 113.537592)
 		(width 0.25)
-		(layer "F.Cu")
+		(layer "B.Cu")
+		(net 74)
+	)
+	(segment
+		(start 159.543884 150.614189)
+		(end 164.430951 150.614189)
+		(width 0.5)
+		(layer "B.Cu")
 		(net 74)
 	)
@@
 	)
 	(segment
-		(start 149.423563 140.493868)
-		(end 149.423563 113.704783)
-		(width 0.5)
-		(layer "B.Cu")
-		(net 77)
-	)
-	(segment
-		(start 164.430951 150.614189)
-		(end 167.95764 147.0875)
-		(width 0.5)
-		(layer "B.Cu")
-		(net 77)
-	)
-	(segment
-		(start 149.423563 140.493868)
-		(end 159.543884 150.614189)
-		(width 0.5)
-		(layer "B.Cu")
-		(net 77)
-	)
-	(segment
-		(start 149.423563 113.704783)
-		(end 149.590754 113.537592)
-		(width 0.5)
-		(layer "B.Cu")
-		(net 77)
-	)
-	(segment
-		(start 149.590754 112.45)
-		(end 149.590754 113.537592)
-		(width 0.25)
-		(layer "B.Cu")
-		(net 77)
-	)
-	(segment
-		(start 159.543884 150.614189)
-		(end 164.430951 150.614189)
-		(width 0.5)
-		(layer "B.Cu")
-		(net 77)
-	)
-	(segment
