File: RKD_06/RKD06_Assemble_Main/RKD06_Assemble_Main.kicad_pcb (KiCad board)
At the start: 2 copper layers, 359.6 x 126.2 mm, 289 parts, among them J1 TRRS, J2 TRRS, J3 Conn_01x04, J4 Qwiic_RA, J5 Qwiic_RA, J6 TRRS, J7 Conn_01x04, J8 TRRS, J9 Conn_01x04, SW1 SW_Push, SW10 SW_Push, SW101 SW_Push, SW102 SW_Push, SW11 SW_Push, SW12 SW_Push, SW13 SW_Push, SW14 SW_Push, SW15 SW_Push, SW16 SW_Push, SW17 SW_Push, SW18 SW_Push, SW19 SW_Push, SW2 SW_Push, SW20 SW_Push, SW21 SW_Push, SW22 SW_Push, SW23 SW_Push, SW24 SW_Push, SW25 SW_Push, SW26 SW_Push, SW27 SW_Push, SW28 SW_Push, SW29 SW_Push, SW3 SW_Push, SW30 SW_Push, SW31 SW_Push, SW32 SW_Push, SW33 SW_Push, SW34 SW_Push, SW35 SW_Push, SW36 SW_Push, SW37 SW_Push, SW38 SW_Push, SW39 SW_Push, SW4 SW_Push, SW40 SW_Push, SW41 SW_Push, SW42 SW_Push, SW5 SW_Push, SW51 SW_Push, SW52 SW_Push, SW53 SW_Push, SW54 SW_Push, SW55 SW_Push, SW56 SW_Push, SW57 SW_Push, SW58 SW_Push, SW59 SW_Push, SW6 SW_Push, SW60 SW_Push, SW61 SW_Push, SW62 SW_Push, SW63 SW_Push, SW64 SW_Push, SW65 SW_Push, SW66 SW_Push, SW67 SW_Push, SW68 SW_Push, SW69 SW_Push, SW7 SW_Push, SW70 SW_Push, SW71 SW_Push, SW72 SW_Push, SW73 SW_Push, SW74 SW_Push, SW75 SW_Push, SW76 SW_Push, SW77 SW_Push, SW78 SW_Push, SW79 SW_Push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

Commit message: 配線
Parts:
- J1, J2: moved to B.Cu
- moved LED37 0.78 mm to (52.4, 42.9)
- turned J1 to 90 degrees
- turned J2 to -90 degrees
Connections:
- J9 pad 1: VCC_R -> VDD_R
Routing:
- net Col0_R: track 0.00 -> 269.1 mm, vias 0 -> 1
- net Col1_R: track 0.00 -> 248.1 mm, vias 0 -> 1
- net Col0_L: track 0.00 -> 238.0 mm, vias 0 -> 1
- net Row4_R: track 0.00 -> 237.3 mm, vias 0 -> 8
- net Col2_R: track 0.00 -> 231.0 mm, vias 0 -> 1
- net GND_R: track 0.00 -> 229.4 mm
- net Row5_R: track 0.00 -> 226.7 mm, vias 0 -> 8
- net Col1_L: track 0.00 -> 225.9 mm, vias 0 -> 1
- net VDD_R: track 0.00 -> 225.8 mm
- net Row5_L: track 0.00 -> 223.0 mm, vias 0 -> 7
- net SDA_R: track 0.00 -> 215.8 mm
- net Col2_L: track 0.00 -> 215.8 mm, vias 0 -> 1
- net Col3_R: track 0.00 -> 213.8 mm, vias 0 -> 1
- net SCL_R: track 0.00 -> 201.9 mm
- net Row4_L: track 0.00 -> 201.3 mm, vias 0 -> 7
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Other:
- board text added: "RKD06 v1.0"

Commit message: RKD-6修正
Parts:
- added REF**: rkd_LOGO_2x, Rikkodo_FootPrint:rkd_LOGO_2x, F.Cu at (207.2, 69.1)
- added Ref**: Val**, kbd_Hole:m2_Spacer_Hole_hex, F.Cu at (154.8, 116.7)
- added Ref**: Val**, kbd_Hole:m2_Spacer_Hole_hex, F.Cu at (300.1, 116.7)
- added Ref**: Val**, kbd_Hole:m2_Spacer_Hole_hex, F.Cu at (323.9, 78.6)
- added Ref**: Val**, kbd_Hole:m2_Spacer_Hole_hex, F.Cu at (102.4, 78.6)
- moved SW101 12.8 mm to (204.8, 35.7), turned to 180 degrees
- moved SW102 12.8 mm to (385.8, 35.7), turned to 180 degrees
- moved J3 12.2 mm to (206.3, 75.9), turned to -90 degrees
- moved J6 11.9 mm to (219.1, 47.6)
- moved J8 11.9 mm to (400.1, 47.6)
- moved R2 2.38 mm to (217.3, 64.0)
- moved R1 2.38 mm to (203.0, 64.0)
Routing:
- net GND_L: track 97.9 -> 125.2 mm
- net VDD_R: track 225.8 -> 238.9 mm
- net VCC_L: track 121.4 -> 132.9 mm
- net SDA_L: track 76.5 -> 85.6 mm
- net LED_R: track 29.2 -> 35.4 mm
- net RST_L: track 4.57 -> 10.3 mm
- net RST_R: track 4.57 -> 10.3 mm
- net Col6_R: track 181.1 -> 176.5 mm
- net LED_L: track 28.3 -> 32.9 mm
- net GND_R: track 229.4 -> 233.9 mm
- net Row2_R: track 168.3 -> 172.7 mm
- net Row2_L: track 162.8 -> 167.2 mm
- net Col4_R: track 195.2 -> 198.1 mm
- net Col3_R: track 213.8 -> 212.7 mm
- net SCL_L: track 69.0 -> 69.5 mm
Other:
- outline, holes or cut-outs redrawn

Commit message: LED位置調整
Parts:
- moved LED28 2.38 mm to (202.4, 90.5)
Changed lines of the file:
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@@
 	(footprint "Rikkodo_FootPrint:rkd_LEDHall"
 		(layer "F.Cu")
-		(at 200.025 90.4875)
+		(at 202.40625 90.4875)
 		(property "Reference" "LED28"
 			(at 0 -2.4 0)

Commit message: 出力先パスを設定
Other:
- board text added: "RKD06_Assemble v1.0"
Changed lines of the file:
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@@
 			(drillshape 0)
 			(scaleselection 1)
-			(outputdirectory "../../../../Order/20241231/RKD01/Assemble_R/")
+			(outputdirectory "../../../Order/20241231/RKD06/Assemble/")
 		)
 	)
@@
 		)
 	)
-	(gr_text "RKD06 v1.0"
-		(at 71.4375 95.25 0)
+	(gr_text "RKD06_Assemble v1.0"
+		(at 69.05625 35.71875 0)
 		(layer "B.SilkS")
 		(effects
