File: RKD_Common/RKD_ORDER_2_0.8mm/RKD_ORDER_2.kicad_pcb (KiCad board)
At the start: 2 copper layers, 66.7 x 81 mm, 22 parts, among them J1 Qwiic_RA, J2 Conn_01x06, J3 Conn_01x24, J4 Qwiic_RA, J5 Conn_01x06, J6 Qwiic_RA, J7 Conn_01x06, M1 Mark, M10 Mark, M11 Mark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

Commit message: ORDER REMAKE
Parts:
- removed M1: Mark, Rikkodo_FootPrint:rkd_Point_Hall
- removed M4: Mark, kbd_Hole:m2_Screw_Hole
- added J10: Conn_01x24, Connector_FFC-FPC:Hirose_FH12-24S-0.5SH_1x24-1MP_P0.50mm_Horizontal, B.Cu at (114.3, 56.0)
- added J8: Qwiic_RA, SparkFun-Connector:JST_SMD_1.0mm-4_Black, B.Cu at (118.7, 42.9)
- added J9: Conn_01x06, Connector_FFC-FPC:Hirose_FH12-6S-0.5SH_1x06-1MP_P0.50mm_Horizontal, B.Cu at (126.2, 82.5)
- added M10: Mark, Rikkodo_FootPrint:rkd_cutdot, F.Cu at (89.6, 86.3)
- added M10: Mark, Rikkodo_FootPrint:rkd_cutdot, F.Cu at (108.0, 68.5)
- added M2: Mark, kbd_Hole:m2_Screw_Hole, F.Cu at (132.2, 113.1)
- added M3: Mark, kbd_Hole:m2_Screw_Hole, F.Cu at (120.3, 113.1)
- added M9: Mark, kbd_Hole:m2_Screw_Hole, F.Cu at (131.0, 53.6)
- added OL2: OLED, BrownSugar_KBD:OLED_center_display, F.Cu at (119.9, 101.2)
- added Picot1: rkd_picot5400_BTM, Rikkodo_FootPrint:rkd_picot5400_BTM, F.Cu at (104.8, 56.0)
- added U2: Pico, Rikkodo_FootPrint:rkd_RPi_Pico_TH_NODBG, F.Cu at (126.2, 90.5)
- moved J4 47.2 mm to (95.0, 91.1)
- moved M5 47.2 mm to (99.4, 98.2)
- moved Trackball1 47.2 mm to (99.4, 98.2)
- moved M11 38.7 mm to (85.4, 72.6)
- moved J7 22.9 mm to (104.8, 65.2), turned to 90 degrees
- moved J6 20.8 mm to (98.2, 47.6), turned to 0 degrees
- moved M6 17.5 mm to (98.2, 56.6), turned to 180 degrees
- moved M7 17.5 mm to (98.2, 56.6), turned to 180 degrees
- moved M8 17.5 mm to (98.2, 56.6), turned to -90 degrees
- moved J5 15.3 mm to (99.4, 56.6), turned to 90 degrees
- turned J2 to -90 degrees
Connections:
- J2 pad 1: GND -> 3v3
- J2 pad 2: SCLK -> GND
- J2 pad 3: SDIO_TX -> unconnected-(J2-Pin_3-Pad3)
- J2 pad 4: unconnected-(J2-Pin_4-Pad4) -> SDIO_TX
- J2 pad 5: GND -> SCLK
- J2 pad 6: 3v3 -> GND
Routing:
- net GND_2: track 0.00 -> 197.6 mm
- net 3v3_2: track 0.00 -> 183.1 mm
- net SCL-Tx_2: track 0.00 -> 78.6 mm
- net SDA-SCK_2: track 0.00 -> 74.9 mm
- net GP18_2: track 0.00 -> 69.4 mm
- net GP17_2: track 0.00 -> 57.6 mm
- net GP16_2: track 0.00 -> 55.6 mm
- net VCC_2: track 0.00 -> 53.1 mm
- net GP19_2: track 0.00 -> 52.4 mm
- net GP20_2: track 0.00 -> 46.3 mm
- net GP08_2: track 0.00 -> 46.0 mm
- net GP09_2: track 0.00 -> 44.1 mm
- net GP21_2: track 0.00 -> 42.8 mm
- net GP10_2: track 0.00 -> 39.6 mm
- net GP11_2: track 0.00 -> 37.6 mm
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Other:
- board size 66.7 x 81 mm -> 82.2 x 81 mm
- board text added: "<-- NO_PCBA"
