File: RKD_Common/RKD_ORDER_2_0.8mm/RKD_ORDER_2.kicad_sch (KiCad schematic)
At the start: 22 parts, among them J1 Qwiic_RA, J2 Conn_01x06, J3 Conn_01x24, J4 Qwiic_RA, J5 Conn_01x06, J6 Qwiic_RA, J7 Conn_01x06, M1 Mark, M10 Mark, M11 Mark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

Commit message: ORDER REMAKE
Parts:
- removed M1: Mark, Rikkodo_FootPrint:rkd_Point_Hall, symbol BrownSugar_KBD:Mark
- removed M2, M3, M4, M9: Mark, kbd_Hole:m2_Screw_Hole, symbol BrownSugar_KBD:Mark
- removed M6: Mark, Rikkodo_FootPrint:rkd_Point_Screw_Hall, symbol BrownSugar_KBD:Mark
- removed M7, M8: rkd_SekiBall_ScrewHall, Rikkodo_FootPrint:rkd_SekiBall_ScrewHall, symbol BrownSugar_KBD:Mark
- removed Picot1: rkd_picot5400_BTM, Rikkodo_FootPrint:rkd_picot5400_BTM, symbol BrownSugar_KBD:Mark
- added J10: Conn_01x24, Connector_FFC-FPC:Hirose_FH12-24S-0.5SH_1x24-1MP_P0.50mm_Horizontal, symbol Connector_Generic:Conn_01x24
- added J8: Qwiic_RA, SparkFun-Connector:JST_SMD_1.0mm-4_Black, symbol SparkFun-Connector:Qwiic_Right_Angle
- added J9: Conn_01x06, Connector_FFC-FPC:Hirose_FH12-6S-0.5SH_1x06-1MP_P0.50mm_Horizontal, symbol Connector_Generic:Conn_01x06
- added OL2: OLED, BrownSugar_KBD:OLED_center_display, symbol BrownSugar_KBD:OLED
- added U2: Pico, Rikkodo_FootPrint:rkd_RPi_Pico_TH_NODBG, symbol RPi_Pico:Pico
Connections:
- net 3v3: now also J2.1 (Pin_1); no longer J2.6 (Pin_6)
- net GND: now also J2.2 (Pin_2), J2.6 (Pin_6); no longer J2.1 (Pin_1), J2.5 (Pin_5)
- net SCLK: now also J2.5 (Pin_5); no longer J2.2 (Pin_2)
- net SDIO_TX: now also J2.4 (Pin_4); no longer J2.3 (Pin_3)
- new net 3v3_2: J10.3 (Pin_3), J8.2 (Pin_2), J9.1 (Pin_1), OL2.3 (VCC), U2.36 (3V3)
- new net GND_2: J10.1 (Pin_1), J8.1 (Pin_1), J9.2 (Pin_2), J9.6 (Pin_6), OL2.4 (GND), U2.13 (GND), U2.18 (GND), U2.23 (GND), U2.28 (GND), U2.3 (GND), U2.38 (GND), U2.8 (GND)
- new net GP08_2: J10.17 (Pin_17), U2.11 (GPIO8)
- new net GP09_2: J10.18 (Pin_18), U2.12 (GPIO9)
- new net GP10_2: J10.19 (Pin_19), U2.14 (GPIO10)
- new net GP11_2: J10.20 (Pin_20), U2.15 (GPIO11)
- new net GP12_2: J10.21 (Pin_21), U2.16 (GPIO12)
- new net GP13_2: J10.22 (Pin_22), U2.17 (GPIO13)
- new net GP14_2: J10.23 (Pin_23), U2.19 (GPIO14)
- new net GP15_2: J10.24 (Pin_24), U2.20 (GPIO15)
- new net GP16_2: J10.16 (Pin_16), U2.7 (GPIO5)
- new net GP17_2: J10.15 (Pin_15), U2.6 (GPIO4)
- new net GP18_2: J10.14 (Pin_14), U2.2 (GPIO1)
- new net GP19_2: J10.13 (Pin_13), U2.34 (GPIO28_ADC2)
- new net GP20_2: J10.12 (Pin_12), U2.32 (GPIO27_ADC1)
- new net GP21_2: J10.11 (Pin_11), U2.31 (GPIO26_ADC0)
- new net GP22_2: J10.10 (Pin_10), U2.29 (GPIO22)
- new net GP23_2: J10.9 (Pin_9), U2.27 (GPIO21)
- new net GP24_2: J10.8 (Pin_8), U2.26 (GPIO20)
- new net GP25_2: J10.7 (Pin_7), U2.25 (GPIO19)
- new net GP26_2: J10.6 (Pin_6), U2.24 (GPIO18)
- new net GP27_2: J10.5 (Pin_5), U2.22 (GPIO17)
- new net GP28_2: J10.4 (Pin_4), U2.21 (GPIO16)
- new net SCL-Tx_2: J8.4 (Pin_4), OL2.2 (SCL), U2.10 (GPIO7)
- new net SCLK_2: J9.5 (Pin_5), U2.4 (GPIO2)
- new net SDA-SCK_2: J8.3 (Pin_3), OL2.1 (SDA), U2.9 (GPIO6)
- new net SDIO_TX_2: J9.4 (Pin_4), U2.5 (GPIO3)
- new net VCC_2: J10.2 (Pin_2), U2.39 (VSYS)
- no-connect marks 12 -> 22
Other:
- moved on the sheet: J5, J6, J7
