File: RKD_05/RKD05_AssembleBO/RKD05_AssembleBO.kicad_pcb (KiCad board)
At the start: 2 copper layers, 361.9 x 100 mm, 153 parts, among them J1 Conn_01x02_Socket, J2 Conn_01x24, J3 Conn_01x24, M1 Mark, M2 Mark, M3 Mark, M4 Mark, M5 Mark, M6 Mark, M7 Mark, M8 Mark, SW1 SW_Push, SW10 SW_Push, SW11 SW_Push, SW12 SW_Push, SW13 SW_Push, SW14 SW_Push, SW15 SW_Push, SW16 SW_Push, SW17 SW_Push, SW18 SW_Push, SW19 SW_Push, SW2 SW_Push, SW20 SW_Push, SW21 SW_Push, SW22 SW_Push, SW23 SW_Push, SW24 SW_Push, SW25 SW_Push, SW26 SW_Push, SW27 SW_Push, SW28 SW_Push, SW29 SW_Push, SW3 SW_Push, SW30 SW_Push, SW4 SW_Push, SW40 RotaryEncoder_Switch, SW5 SW_Push, SW51 SW_Push, SW52 SW_Push, SW53 SW_Push, SW54 SW_Push, SW55 SW_Push, SW56 SW_Push, SW57 SW_Push, SW58 SW_Push, SW59 SW_Push, SW6 SW_Push, SW60 SW_Push, SW61 SW_Push, SW62 SW_Push, SW63 SW_Push, SW64 SW_Push, SW65 SW_Push, SW66 SW_Push, SW67 SW_Push, SW68 SW_Push, SW69 SW_Push, SW7 SW_Push, SW70 SW_Push, SW71 SW_Push, SW72 SW_Push, SW73 SW_Push, SW74 SW_Push, SW75 SW_Push, SW76 SW_Push, SW77 SW_Push, SW78 SW_Push, SW79 SW_Push, SW8 SW_Push, SW80 SW_Push, SW81 SW_Push, SW82 SW_Push, SW83 SW_Push, SW84 SW_Push, SW85 SW_Push, SW86 SW_Push, SW87 SW_Push, SW88 SW_Push, SW89 SW_Push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

Commit message: 微調整
Routing:
- net GP11:COL10: track 236.3 -> 234.5 mm
- net GP10:COL11: track 257.1 -> 256.1 mm
Other:
- outline, holes or cut-outs redrawn
Changed lines of the file:
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@@
 	)
 	(gr_line
-		(start 179.784375 133.35)
-		(end 186.928125 126.20625)
+		(start 178.59375 133.35)
+		(end 185.7375 126.20625)
 		(stroke
 			(width 0.05)
@@
 	)
 	(gr_line
-		(start 198.834375 126.20625)
-		(end 205.978125 133.35)
+		(start 200.025 126.20625)
+		(end 207.16875 133.35)
 		(stroke
 			(width 0.05)
@@
 	)
 	(gr_line
-		(start 186.928125 126.20625)
-		(end 198.834375 126.20625)
+		(start 185.7375 126.20625)
+		(end 200.025 126.20625)
 		(stroke
 			(width 0.05)
@@
 	)
 	(gr_line
-		(start 205.978125 133.35)
+		(start 207.16875 133.35)
 		(end 211.93125 133.35)
 		(stroke
@@
 	(gr_line
 		(start 173.83125 133.35)
-		(end 179.784375 133.35)
+		(end 178.59375 133.35)
 		(stroke
 			(width 0.05)
@@
 	)
 	(segment
-		(start 186.928282 107.141496)
-		(end 186.928282 107.126496)
+		(start 186.928282 108.822967)
+		(end 194.548039 101.20321)
 		(width 0.25)
 		(layer "F.Cu")
@@
 	)
 	(segment
-		(start 192.851568 101.20321)
+		(start 194.548039 101.20321)
 		(end 307.754687 101.20321)
 		(width 0.25)
@@
 		(net 84)
 	)
-	(segment
-		(start 186.928282 107.126496)
-		(end 192.851568 101.20321)
-		(width 0.25)
-		(layer "F.Cu")
-		(net 84)
-	)
 	(via
-		(at 186.928282 107.141496)
+		(at 186.928282 108.822967)
 		(size 0.6)
 		(drill 0.3)
@@
 	)
 	(segment
-		(start 186.928282 108.822967)
-		(end 170.735625 125.015624)
-		(width 0.25)
-		(layer "B.Cu")
-		(net 84)
-	)
-	(segment
 		(start 322.6375 148.775)
 		(end 327.4 153.5375)
@@
 	)
 	(segment
-		(start 186.928282 107.141496)
-		(end 186.928282 108.822967)
+		(start 317.875 129.725)
+		(end 322.6375 134.4875)
 		(width 0.25)
 		(layer "B.Cu")
@@
 	)
 	(segment
-		(start 317.875 129.725)
-		(end 322.6375 134.4875)
+		(start 186.928282 108.822967)
+		(end 170.735625 125.015624)
 		(width 0.25)
 		(layer "B.Cu")
@@
 	)
 	(segment
-		(start 193.44688 101.798523)
-		(end 288.704687 101.798523)
+		(start 288.704687 101.798523)
+		(end 289.3 102.393836)
 		(width 0.25)
 		(layer "F.Cu")
@@
 	)
 	(segment
-		(start 188.11875 107.126653)
-		(end 193.44688 101.798523)
+		(start 188.11875 110.172499)
+		(end 196.492726 101.798523)
 		(width 0.25)
 		(layer "F.Cu")
@@
 	)
 	(segment
-		(start 288.704687 101.798523)
-		(end 289.3 102.393836)
+		(start 196.492726 101.798523)
+		(end 288.704687 101.798523)
 		(width 0.25)
 		(layer "F.Cu")
@@
 	)
 	(via
-		(at 188.11875 107.126653)
+		(at 188.11875 110.172499)
 		(size 0.6)
 		(drill 0.3)
@@
 	)
 	(segment
-		(start 188.11875 107.126653)
-		(end 188.11875 110.172499)
-		(width 0.25)
-		(layer "B.Cu")
-		(net 85)
-	)
-	(segment
 		(start 289.3 102.393836)
 		(end 289.3 110.675)
@@
 	)
 	(segment
-		(start 202.699185 98.477)
-		(end 201.402435 97.18025)
+		(start 254.79375 97.63125)
+		(end 253.948 98.477)
 		(width 0.25)
 		(layer "B.Cu")
@@
 	)
 	(segment
-		(start 360.7375 115.4375)
-		(end 360.7375 129.725)
+		(start 355.975 102.966975)
+		(end 347.662792 94.654767)
 		(width 0.25)
 		(layer "B.Cu")
@@
 	)
 	(segment
-		(start 295.32705 97.63125)
-		(end 254.79375 97.63125)
+		(start 360.7375 115.4375)
+		(end 360.7375 129.725)
 		(width 0.25)
 		(layer "B.Cu")
@@
 	)
 	(segment
-		(start 171.737904 119.935624)
-		(end 170.735625 119.935624)
+		(start 214.615141 98.477)
+		(end 203.570861 98.477)
 		(width 0.25)
 		(layer "B.Cu")
@@
 	)
 	(segment
-		(start 313.98681 96.8322)
-		(end 312.24526 98.57375)
+		(start 203.570861 98.477)
+		(end 202.274111 97.18025)
 		(width 0.25)
 		(layer "B.Cu")
@@
 	)
 	(segment
-		(start 334.176 96.8322)
-		(end 313.98681 96.8322)
+		(start 366.117495 167.207505)
+		(end 365.5 167.825)
 		(width 0.25)
 		(layer "B.Cu")
@@
 	)
 	(segment
-		(start 336.353433 94.654767)
-		(end 334.176 96.8322)
+		(start 334.176 96.8322)
+		(end 313.98681 96.8322)
 		(width 0.25)
 		(layer "B.Cu")
@@
 	)
 	(segment
-		(start 254.79375 97.63125)
-		(end 253.948 98.477)
+		(start 372.9875 139.625)
+		(end 373.85625 139.625)
 		(width 0.25)
 		(layer "B.Cu")
@@
 	)
 	(segment
-		(start 366.117495 167.207505)
-		(end 365.5 167.825)
+		(start 202.274111 97.18025)
+		(end 194.493278 97.18025)
 		(width 0.25)
 		(layer "B.Cu")
@@
 	)
 	(segment
-		(start 242.092873 97.180332)
-		(end 215.911809 97.180332)
+		(start 253.948 98.477)
+		(end 243.389541 98.477)
 		(width 0.25)
 		(layer "B.Cu")
@@
 	)
 	(segment
-		(start 253.948 98.477)
-		(end 243.389541 98.477)
+		(start 347.662792 94.654767)
+		(end 336.353433 94.654767)
 		(width 0.25)
 		(layer "B.Cu")
@@
 	)
 	(segment
-		(start 372.9875 139.625)
-		(end 373.85625 139.625)
+		(start 355.975 110.675)
+		(end 360.7375 115.4375)
 		(width 0.25)
 		(layer "B.Cu")
@@
 	)
 	(segment
-		(start 355.975 110.675)
-		(end 355.975 102.966975)
+		(start 312.24526 98.57375)
+		(end 296.26955 98.57375)
 		(width 0.25)
 		(layer "B.Cu")
@@
 	)
 	(segment
-		(start 296.26955 98.57375)
-		(end 295.32705 97.63125)
+		(start 171.737904 119.935624)
+		(end 170.735625 119.935624)
 		(width 0.25)
 		(layer "B.Cu")
@@
 	)
 	(segment
-		(start 355.975 110.675)
-		(end 360.7375 115.4375)
+		(start 365.5 167.825)
+		(end 365.5 186.875)
 		(width 0.25)
 		(layer "B.Cu")
@@
 	)
 	(segment
-		(start 214.615141 98.477)
-		(end 202.699185 98.477)
+		(start 336.353433 94.654767)
+		(end 334.176 96.8322)
 		(width 0.25)
 		(layer "B.Cu")
@@
 	)
 	(segment
-		(start 355.975 102.966975)
-		(end 347.662792 94.654767)
+		(start 355.975 110.675)
+		(end 355.975 102.966975)
 		(width 0.25)
 		(layer "B.Cu")
@@
 	)
 	(segment
-		(start 365.5 167.825)
-		(end 365.5 186.875)
+		(start 366.117495 132.754995)
+		(end 366.117495 167.207505)
 		(width 0.25)
 		(layer "B.Cu")
@@
 	)
 	(segment
-		(start 312.24526 98.57375)
-		(end 296.26955 98.57375)
+		(start 242.092873 97.180332)
+		(end 215.911809 97.180332)
 		(width 0.25)
 		(layer "B.Cu")
@@
 	)
 	(segment
-		(start 194.493278 97.18025)
-		(end 171.737904 119.935624)
+		(start 215.911809 97.180332)
+		(end 214.615141 98.477)
 		(width 0.25)
 		(layer "B.Cu")
@@
 	)
 	(segment
-		(start 201.402435 97.18025)
-		(end 194.493278 97.18025)
+		(start 295.32705 97.63125)
+		(end 254.79375 97.63125)
 		(width 0.25)
 		(layer "B.Cu")
@@
 	)
 	(segment
-		(start 366.117495 132.754995)
-		(end 366.117495 167.207505)
+		(start 313.98681 96.8322)
+		(end 312.24526 98.57375)
 		(width 0.25)
 		(layer "B.Cu")
@@
 	)
 	(segment
-		(start 215.911809 97.180332)
-		(end 214.615141 98.477)
+		(start 296.26955 98.57375)
+		(end 295.32705 97.63125)
 		(width 0.25)
 		(layer "B.Cu")
@@
 	)
 	(segment
-		(start 347.662792 94.654767)
-		(end 336.353433 94.654767)
+		(start 363.0875 129.725)
+		(end 372.9875 139.625)
 		(width 0.25)
 		(layer "B.Cu")
@@
 	)
 	(segment
-		(start 363.0875 129.725)
-		(end 372.9875 139.625)
+		(start 194.493278 97.18025)
+		(end 171.737904 119.935624)
 		(width 0.25)
 		(layer "B.Cu")
@@
 	)
 	(segment
-		(start 155.495625 114.855624)
-		(end 159.404745 118.764744)
+		(start 154.281751 111.227624)
+		(end 156.471374 111.227624)
 		(width 0.25)
 		(layer "F.Cu")
@@
 	)
 	(segment
-		(start 154.281751 111.227624)
-		(end 156.471374 111.227624)
+		(start 314.325 153.0062)
+		(end 333.375 153.0062)
 		(width 0.25)
 		(layer "F.Cu")
@@
 	)
 	(segment
-		(start 314.325 153.0062)
-		(end 333.375 153.0062)
+		(start 159.404745 118.764744)
+		(end 199.48716 118.764744)
 		(width 0.25)
 		(layer "F.Cu")
@@
 	)
 	(segment
+		(start 155.495625 114.855624)
+		(end 159.404745 118.764744)
+		(width 0.25)
+		(layer "F.Cu")
+		(net 95)
+	)
+	(segment
 		(start 156.471374 111.227624)
 		(end 157.1625 111.91875)
@@
 	)
 	(segment
+		(start 199.48716 118.764744)
+		(end 213.362499 132.640083)
+		(width 0.25)
+		(layer "F.Cu")
+		(net 95)
+	)
+	(segment
 		(start 119.0625 153.0062)
 		(end 119.073259 152.995441)
@@
 	)
 	(segment
-		(start 159.404745 118.764744)
-		(end 199.48716 118.764744)
+		(start 213.362499 147.293699)
+		(end 219.075 153.0062)
 		(width 0.25)
 		(layer "F.Cu")
@@
 	)
 	(segment
-		(start 213.6875 132.965084)
-		(end 213.6875 147.6187)
-		(width 0.25)
-		(layer "F.Cu")
-		(net 95)
-	)
-	(segment
-		(start 213.6875 147.6187)
-		(end 219.075 153.0062)
-		(width 0.25)
-		(layer "F.Cu")
-		(net 95)
-	)
-	(segment
 		(start 102.1813 155.175)
 		(end 100.0125 153.0062)
@@
 	)
 	(segment
-		(start 157.1625 111.91875)
-		(end 157.1625 113.188749)
+		(start 213.362499 132.640083)
+		(end 213.362499 147.293699)
 		(width 0.25)
 		(layer "F.Cu")
@@
 	)
 	(segment
-		(start 295.275 153.0062)
-		(end 314.325 153.0062)
+		(start 157.1625 111.91875)
+		(end 157.1625 113.188749)
 		(width 0.25)
 		(layer "F.Cu")
@@
 	)
 	(segment
-		(start 199.48716 118.764744)
-		(end 213.6875 132.965084)
+		(start 295.275 153.0062)
+		(end 314.325 153.0062)
 		(width 0.25)
 		(layer "F.Cu")
