File: RKD_04/RKD04_Top/RKD04_Top.kicad_pcb (KiCad board)
At the start: 2 copper layers, 97.6 x 97.6 mm, 19 parts, among them SW1 RotaryEncoder_Switch, SW10 SW_Push, SW11 SW_Push, SW12 SW_Push, SW13 SW_Push, SW14 SW_Push, SW2 RotaryEncoder_Switch, SW3 RotaryEncoder_Switch, SW4 RotaryEncoder_Switch, SW5 SW_Push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

Commit message: 追加
Parts:
- added REF**: rkd_LOGO_2x, Rikkodo_FootPrint:rkd_LOGO_2x, F.Cu at (54.8, 28.6)
- moved SW8 2.38 mm to (71.4, 104.8)
- moved SW14 2.38 mm to (128.6, 104.8)
Other:
- outline, holes or cut-outs redrawn
Changed lines of the file:
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@@
 	(footprint "kbd_SW_Hole:SW_Hole_1u"
 		(layer "F.Cu")
-		(at 69.056148 104.774937)
+		(at 71.4375 104.774937)
 		(property "Reference" "SW8"
 			(at 7 8.1 0)
@@
 		(embedded_fonts no)
 	)
+	(footprint "Rikkodo_FootPrint:rkd_LOGO_2x"
+		(layer "F.Cu")
+		(at 54.76875 28.575)
+		(property "Reference" "REF**"
+			(at 0 -0.5 0)
+			(unlocked yes)
+			(layer "F.SilkS")
+			(hide yes)
+			(effects
+				(font
+					(size 1 1)
+					(thickness 0.1)
+				)
+			)
+		)
+		(property "Value" "rkd_LOGO_2x"
+			(at 0 1 0)
+			(unlocked yes)
+			(layer "F.Fab")
+			(hide yes)
+			(effects
+				(font
+					(size 1 1)
+					(thickness 0.15)
+				)
+			)
+		)
+		(property "Datasheet" ""
+			(at 0 0 0)
+			(unlocked yes)
+			(layer "F.Fab")
+			(hide yes)
+			(effects
+				(font
+					(size 1 1)
+					(thickness 0.15)
+				)
+			)
+		)
+		(property "Description" ""
+			(at 0 0 0)
+			(unlocked yes)
+			(layer "F.Fab")
+			(hide yes)
+			(effects
+				(font
+					(size 1 1)
+					(thickness 0.15)
+				)
+			)
+		)
+		(attr smd board_only exclude_from_pos_files exclude_from_bom)
+		(fp_line
+			(start -5.155554 -2.97656)
+			(end -5.155554 2.97656)
+			(stroke
+				(width 0.25)
+				(type default)
+			)
+			(layer "F.SilkS")
+		)
+		(fp_line
+			(start -5.155554 -2.97656)
+			(end 0 0)
+			(stroke
+				(width 0.25)
+				(type default)
+			)
+			(layer "F.SilkS")
+		)
+		(fp_line
+			(start -5.155554 2.97656)
+			(end 0 5.95312)
+			(stroke
+				(width 0.25)
+				(type default)
+			)
+			(layer "F.SilkS")
+		)
+		(fp_line
+			(start -2.577777 -1.48828)
+			(end -2.577777 4.46484)
+			(stroke
+				(width 0.25)
+				(type default)
+			)
+			(layer "F.SilkS")
+		)
+		(fp_line
+			(start 0 -5.95312)
+			(end -5.155554 -2.97656)
+			(stroke
+				(width 0.25)
+				(type default)
+			)
+			(layer "F.SilkS")
+		)
+		(fp_line
+			(start 0 -5.95312)
+			(end 0 0)
+			(stroke
+				(width 0.25)
+				(type default)
+			)
+			(layer "F.SilkS")
+		)
+		(fp_line
+			(start 0 -5.95312)
+			(end 5.155554 -2.97656)
+			(stroke
+				(width 0.25)
+				(type default)
+			)
+			(layer "F.SilkS")
+		)
+		(fp_line
+			(start 0 5.95312)
+			(end 5.155554 2.97656)
+			(stroke
+				(width 0.25)
+				(type default)
+			)
+			(layer "F.SilkS")
+		)
+		(fp_line
+			(start 2.577777 -1.48828)
+			(end 2.577777 4.46484)
+			(stroke
+				(width 0.25)
+				(type default)
+			)
+			(layer "F.SilkS")
+		)
+		(fp_line
+			(start 5.155554 -2.97656)
+			(end 0 0)
+			(stroke
+				(width 0.25)
+				(type default)
+			)
+			(layer "F.SilkS")
+		)
+		(fp_line
+			(start 5.155554 -2.97656)
+			(end 5.155554 2.97656)
+			(stroke
+				(width 0.25)
+				(type default)
+			)
+			(layer "F.SilkS")
+		)
+		(embedded_fonts no)
+	)
 	(footprint "kbd_SW_Hole:SW_Hole_1u"
 		(layer "F.Cu")
@@
 	(footprint "kbd_SW_Hole:SW_Hole_1u"
 		(layer "F.Cu")
-		(at 130.968648 104.774987)
+		(at 128.5875 104.774987)
 		(property "Reference" "SW14"
 			(at 7 8.1 0)
@@
 		(layer "Edge.Cuts")
 	)
-	(gr_line
-		(start 90.487576 36.909406)
-		(end 48.815666 36.909406)
-		(stroke
-			(width 0.05)
-			(type default)
-		)
-		(layer "Edge.Cuts")
-	)
-	(gr_line
-		(start 90.487577 17.85939)
-		(end 90.487576 36.909406)
+	(gr_arc
+		(start 42.8625 17.859375)
+		(mid 43.21563 17.013094)
+		(end 44.065541 16.668792)
 		(stroke
 			(width 0.05)
@@
 		(layer "Edge.Cuts")
 	)
-	(gr_arc
-		(start 90.487577 17.85939)
-		(mid 90.836303 17.017491)
-		(end 91.678202 16.668765)
-		(stroke
-			(width 0.05)
-			(type default)
-		)
-		(layer "Edge.Cuts")
-	)
-	(gr_arc
-		(start 42.8625 17.859375)
-		(mid 43.211226 17.017476)
-		(end 44.053125 16.66875)
-		(stroke
-			(width 0.05)
-			(type default)
-		)
-		(layer "Edge.Cuts")
-	)
 	(gr_line
 		(start 140.4938 27.384375)
 		(end 140.49375 113.109375)
-		(stroke
-			(width 0.05)
-			(type default)
-		)
-		(layer "Edge.Cuts")
-	)
-	(gr_line
-		(start 48.815666 36.909406)
-		(end 48.815666 17.85939)
 		(stroke
 			(width 0.05)
@@
 	)
 	(gr_line
-		(start 47.62504 16.668765)
-		(end 44.053125 16.66875)
-		(stroke
-			(width 0.05)
-			(type default)
-		)
-		(layer "Edge.Cuts")
-	)
-	(gr_line
 		(start 79.390608 38.646049)
 		(end 79.390608 41.721049)
@@
 	(gr_line
 		(start 98.821875 16.66875)
-		(end 91.678202 16.668765)
+		(end 44.06554 16.668865)
 		(stroke
 			(width 0.05)
@@
 		(stroke
 			(width 0.05)
-			(type default)
-		)
-		(layer "Edge.Cuts")
-	)
-	(gr_arc
-		(start 47.62504 16.668765)
-		(mid 48.466939 17.017491)
-		(end 48.815665 17.85939)
-		(stroke
-			(width 0.05)
