File: RKD_07/RKD07_ReMecab/RKD07_ReMecab.kicad_pcb (KiCad board)
At the start: 2 copper layers, 70.8 x 98.2 mm, 35 parts, among them J13 Conn_01x04, J2 Conn_01x24, J3 Qwiic_RA, J4 Conn_01x06, J5 Conn_01x02_Socket, J7 Conn_01x08, J8 Conn_01x06, SW41 SW_Push, U1 Pico

Commit message: 07 Rebuild
Parts:
- moved R5 9.84 mm to (103.6, 44.6), turned to 180 degrees
- turned R6 to 180 degrees
Routing:
- net CS: track 21.1 -> 14.0 mm
- net GND: track 178.5 -> 177.8 mm, vias 20 -> 22
Other:
- board text added: "03 02 00"
- board text removed: "03 02 01"

Commit message: 調整
Parts:
- removed the REF** at (112.5, 64.6)
- added REF**: rkd_cutdot_no_edgecut_16, Rikkodo_FootPrint:rkd_cutdot_no_edgecut_16, F.Cu at (123.2, 64.6)
- added REF**: rkd_cutdot_no_edgecut_4, Rikkodo_FootPrint:rkd_cutdot_no_edgecut_4, F.Cu at (106.6, 64.6)
- added REF**: rkd_cutdot_no_edgecut_4, Rikkodo_FootPrint:rkd_cutdot_no_edgecut_4, F.Cu at (101.8, 64.6)
- added REF**: rkd_cutdot_no_edgecut_4, Rikkodo_FootPrint:rkd_cutdot_no_edgecut_4, F.Cu at (111.3, 64.6)
- added REF**: rkd_cutdot_no_edgecut_1, Rikkodo_FootPrint:rkd_cutdot_no_edgecut_1, F.Cu at (97.6, 64.6)
- added Ref**: Val**, kbd_Hole:m3_Screw_Hole_EdgeCuts, F.Cu at (121.4, 57.1)
- added Ref**: Val**, kbd_Hole:m3_Screw_Hole_EdgeCuts, F.Cu at (140.5, 102.4)
- added Ref**: Val**, kbd_Hole:m3_Screw_Hole_EdgeCuts, F.Cu at (138.1, 88.1)
- added Ref**: Val**, kbd_Hole:m3_Screw_Hole_EdgeCuts, F.Cu at (95.2, 64.3)
- moved REF** 33.3 mm to (98.8, 64.6)
- moved J4 1.19 mm to (139.3, 95.2)
Routing:
- net GND: track 177.8 -> 173.6 mm
- net COL5_L: track 119.0 -> 117.3 mm
- net SDA/SCK_L: track 150.4 -> 151.9 mm
- net ROW4_L: track 112.7 -> 114.1 mm
- net SCL/TX_L: track 152.3 -> 151.1 mm

Commit message: Update Remecab
Parts:
- removed J13: Conn_01x04, Connector_PinHeader_2.54mm:PinHeader_1x04_P2.54mm_Horizontal
- removed the REF** at (132.2, 102.1)
- removed the Ref** at (121.4, 57.1)
- removed the Ref** at (140.5, 102.4)
- removed the Ref** at (138.1, 88.1)
- removed the Ref** at (95.2, 64.3)
- added REF**: rkd_cutdot_no_edgecut_1, Rikkodo_FootPrint:rkd_cutdot_no_edgecut_1, F.Cu at (113.1, 107.2)
- added REF**: rkd_cutdot_no_edgecut_1, Rikkodo_FootPrint:rkd_cutdot_no_edgecut_1, F.Cu at (92.6, 105.1)
- added REF**: rkd_cutdot_no_edgecut_1, Rikkodo_FootPrint:rkd_cutdot_no_edgecut_1, F.Cu at (96.4, 64.3)
- added REF**: rkd_cutdot_no_edgecut_1, Rikkodo_FootPrint:rkd_cutdot_no_edgecut_1, F.Cu at (95.2, 64.3)
- added REF**: rkd_cutdot_no_edgecut_1, Rikkodo_FootPrint:rkd_cutdot_no_edgecut_1, F.Cu at (148.2, 64.3)
- added REF**: rkd_cutdot_no_edgecut_1, Rikkodo_FootPrint:rkd_cutdot_no_edgecut_1, F.Cu at (103.9, 106.3)
- added REF**: rkd_cutdot_no_edgecut_4, Rikkodo_FootPrint:rkd_cutdot_no_edgecut_4, F.Cu at (140.5, 64.3)
- added REF**: rkd_cutdot_no_edgecut_1, Rikkodo_FootPrint:rkd_cutdot_no_edgecut_1, F.Cu at (145.9, 64.3)
- added REF**: rkd_cutdot_no_edgecut_1, Rikkodo_FootPrint:rkd_cutdot_no_edgecut_1, F.Cu at (92.6, 103.9)
- added REF**: rkd_cutdot_no_edgecut_1, Rikkodo_FootPrint:rkd_cutdot_no_edgecut_1, F.Cu at (133.1, 105.1)
- added REF**: rkd_cutdot_no_edgecut_16, Rikkodo_FootPrint:rkd_cutdot_no_edgecut_16, F.Cu at (101.8, 107.2)
- added REF**: rkd_cutdot_no_edgecut_1, Rikkodo_FootPrint:rkd_cutdot_no_edgecut_1, F.Cu at (133.1, 64.6)
- added REF**: rkd_cutdot_no_edgecut_1, Rikkodo_FootPrint:rkd_cutdot_no_edgecut_1, F.Cu at (144.7, 64.3)
- added REF**: rkd_cutdot_no_edgecut_1, Rikkodo_FootPrint:rkd_cutdot_no_edgecut_1, F.Cu at (111.9, 107.2)
- added REF**: rkd_cutdot_no_edgecut_1, Rikkodo_FootPrint:rkd_cutdot_no_edgecut_1, F.Cu at (149.4, 64.3)
- added REF**: rkd_cutdot_no_edgecut_1, Rikkodo_FootPrint:rkd_cutdot_no_edgecut_1, F.Cu at (103.9, 103.9)
- added REF**: rkd_cutdot_no_edgecut_1, Rikkodo_FootPrint:rkd_cutdot_no_edgecut_1, F.Cu at (147.0, 64.3)
- added REF**: rkd_cutdot_no_edgecut_1, Rikkodo_FootPrint:rkd_cutdot_no_edgecut_1, F.Cu at (92.6, 106.3)
- added REF**: rkd_cutdot_no_edgecut_1, Rikkodo_FootPrint:rkd_cutdot_no_edgecut_1, F.Cu at (94.1, 64.3)
- added REF**: rkd_cutdot_no_edgecut_1, Rikkodo_FootPrint:rkd_cutdot_no_edgecut_1, F.Cu at (103.9, 105.1)
- added REF**: rkd_cutdot_no_edgecut_1, Rikkodo_FootPrint:rkd_cutdot_no_edgecut_1, F.Cu at (133.1, 103.9)
- added REF**: rkd_cutdot_no_edgecut_1, Rikkodo_FootPrint:rkd_cutdot_no_edgecut_1, F.Cu at (133.1, 106.3)
- added REF**: rkd_cutdot_no_edgecut_1, Rikkodo_FootPrint:rkd_cutdot_no_edgecut_1, F.Cu at (143.5, 64.3)
- added REF**: rkd_cutdot_no_edgecut_1, Rikkodo_FootPrint:rkd_cutdot_no_edgecut_1, F.Cu at (114.3, 107.2)
- added REF**: rkd_cutdot_no_edgecut_4, Rikkodo_FootPrint:rkd_cutdot_no_edgecut_4, F.Cu at (135.7, 64.3)
- added REF**: rkd_cutdot_no_edgecut_1, Rikkodo_FootPrint:rkd_cutdot_no_edgecut_1, F.Cu at (115.5, 107.2)
- added REF**: rkd_cutdot_no_edgecut_1, Rikkodo_FootPrint:rkd_cutdot_no_edgecut_1, F.Cu at (92.6, 64.6)
- added Ref**: Val**, kbd_Hole:m2_Screw_Hole, F.Cu at (102.4, 96.4)
- moved J4 42.6 mm to (123.8, 55.6)
- moved R4 24.5 mm to (132.7, 50.0)
- moved J3 24.3 mm to (134.6, 55.7), turned to 180 degrees
- moved R3 20.5 mm to (132.7, 51.8)
- moved REF** 20.4 mm to (103.9, 83.6), turned to 90 degrees
- moved REF** 10.8 mm to (103.9, 103.0), turned to 90 degrees
- moved REF** 0.89 mm to (133.1, 84.2)
- moved REF** 0.89 mm to (92.6, 84.2)
- moved REF** 0.30 mm to (101.8, 64.3)
- moved REF** 0.30 mm to (97.6, 64.3)
- moved REF** 0.30 mm to (98.8, 64.3)
- moved REF** 0.30 mm to (93.2, 64.3)
- moved REF** 0.30 mm to (111.3, 64.3)
- moved REF** 0.30 mm to (123.2, 64.3)
- moved REF** 0.30 mm to (106.6, 64.3)
Routing:
- net SCL/TX_L: track 151.1 -> 74.1 mm
- net SDA/SCK_L: track 151.9 -> 76.5 mm
- net GND: track 173.6 -> 137.3 mm, vias 22 -> 23
- net 3V3: track 214.4 -> 184.5 mm
- net ROW4_L: track 114.1 -> 122.5 mm
- net COL5_L: track 117.3 -> 125.2 mm
- net VCC: track 85.7 -> 85.0 mm
- net GP00: track 30.8 -> 31.5 mm
Other:
- outline, holes or cut-outs redrawn
- board text added: "3V3 00 CS X 02 SDIO 03 SCLK GND"
- board text added: "VC 3V PD"
- board text removed: "3V3 CS X SDIO SCLK GND"
- board text removed: "Picot5400"
- board text removed: "VC 3V CS"
- board text removed: "VC SC SD GN"

Commit message: ReMecabu
Parts:
- removed D41: D, kbd_Parts:Diode_SMD
- removed J7: Conn_01x08, Connector_PinHeader_2.54mm:PinHeader_1x08_P2.54mm_Horizontal
- removed the REF** at (113.1, 107.2)
- removed the REF** at (101.8, 107.2)
- removed the REF** at (111.9, 107.2)
- removed the REF** at (114.3, 107.2)
- removed the REF** at (115.5, 107.2)
- removed the Ref** at (81.0, 123.8)
- removed the Ref** at (90.5, 123.8)
- removed SW41: SW_Push, Rikkodo_FootPrint:rkd_Asm_ChocV1V2_Hotswap_1u
- added J1: Conn_01x12, Connector_PinHeader_2.54mm:PinHeader_1x12_P2.54mm_Horizontal, B.Cu at (94.7, 51.2)
- moved J4 5.37 mm to (129.2, 56.0)
- moved J3 3.49 mm to (138.1, 56.0)
- moved R3 3.49 mm to (136.2, 52.1)
- moved R4 3.49 mm to (136.2, 50.3)
Routing:
- net COL5_L: track 125.2 -> 10.0 mm
- net ROW4_L: track 122.5 -> 18.9 mm
- net SCL/TX_L: track 74.1 -> 93.1 mm
- net SDA/SCK_L: track 76.5 -> 86.7 mm
- net Net-(D41-A): track 7.17 -> 0.00 mm
- net VCC: track 85.0 -> 90.6 mm
- net GND: track 137.3 -> 132.1 mm, vias 23 -> 15
- net 3V3: track 184.5 -> 186.4 mm
Other:
- board size 70.8 x 98.2 mm -> 70.8 x 78.9 mm
- board text added: "3V3"
- board text added: "GND"
- board text added: "SD SC PD"
- board text added: "VCC"
- board text removed: "GN GN"
- board text removed: "VC 3V PD"
