File: RKD_07/RKD07_ReMecab/RKD07_ReMecab.kicad_sch (KiCad schematic)
At the start: 16 parts, among them J2 Conn_01x24, J3 Qwiic_RA, J4 Conn_01x06, J5 Conn_01x02_Socket, J7 Conn_01x08, J8 Conn_01x06, SW41 SW_Push, U1 Pico

Commit message: ReMecabu
Parts:
- removed D41: D, kbd_Parts:Diode_SMD, symbol Device:D
- removed J7: Conn_01x08, Connector_PinHeader_2.54mm:PinHeader_1x08_P2.54mm_Horizontal, symbol Connector_Generic:Conn_01x08
- removed SW41: SW_Push, Rikkodo_FootPrint:rkd_Asm_ChocV1V2_Hotswap_1u, symbol Switch:SW_Push
- added J1: Conn_01x12, Connector_PinHeader_2.54mm:PinHeader_1x12_P2.54mm_Horizontal, symbol Connector_Generic:Conn_01x12
Connections:
- net 3V3: now also J1.10 (Pin_10), J1.9 (Pin_9)
- net CS: now also J1.6 (Pin_6)
- net GND: now also J1.1 (Pin_1), J1.2 (Pin_2)
- net GP00: now also J1.3 (Pin_3)
- net GP02: now also J1.4 (Pin_4)
- net GP03: now also J1.5 (Pin_5)
- net SCL/TX_L: now also J1.7 (Pin_7)
- net SDA/SCK_L: now also J1.8 (Pin_8)
- net VCC: now also J1.11 (Pin_11), J1.12 (Pin_12)
