File: RKD_08/RKD08_Assmenble/RKD08_Assmenble.kicad_pcb (KiCad board)
At the start: 2 copper layers, 57.7 x 38.7 mm, 40 parts, among them J1 Conn_01x06, J3 Qwiic_RA, SW1 SW_Push, SW2 KEY_SWITCH, U1 ProMicro

Commit message: edit meishi
Parts:
- added ?: , , B.Cu at (92.0, 59.2)
- added REF**: rkd_cutdot_no_edgecut_1, Rikkodo_FootPrint:rkd_cutdot_no_edgecut_1, F.Cu at (78.3, 58.3)
- added REF**: rkd_cutdot_no_edgecut_1, Rikkodo_FootPrint:rkd_cutdot_no_edgecut_1, F.Cu at (131.0, 73.5)
- added REF**: rkd_cutdot_no_edgecut_1, Rikkodo_FootPrint:rkd_cutdot_no_edgecut_1, F.Cu at (92.3, 59.2)
- added REF**: rkd_cutdot_no_edgecut_1, Rikkodo_FootPrint:rkd_cutdot_no_edgecut_1, F.Cu at (88.4, 54.8)
- added REF**: rkd_cutdot_no_edgecut_1, Rikkodo_FootPrint:rkd_cutdot_no_edgecut_1, F.Cu at (78.3, 57.1)
- added REF**: rkd_cutdot_no_edgecut_1, Rikkodo_FootPrint:rkd_cutdot_no_edgecut_1, F.Cu at (89.9, 59.2)
- added REF**: rkd_cutdot_no_edgecut_1, Rikkodo_FootPrint:rkd_cutdot_no_edgecut_1, F.Cu at (76.8, 59.2)
- added REF**: rkd_cutdot_no_edgecut_1, Rikkodo_FootPrint:rkd_cutdot_no_edgecut_1, F.Cu at (78.3, 56.0)
- added REF**: rkd_cutdot_no_edgecut_1_2, Rikkodo_FootPrint:rkd_cutdot_no_edgecut_1_2, F.Cu at (93.2, 54.5)
- added REF**: rkd_cutdot_no_edgecut_1, Rikkodo_FootPrint:rkd_cutdot_no_edgecut_1, F.Cu at (78.3, 54.8)
- added REF**: rkd_cutdot_no_edgecut_1, Rikkodo_FootPrint:rkd_cutdot_no_edgecut_1, F.Cu at (78.0, 59.2)
- added REF**: rkd_cutdot_no_edgecut_4, Rikkodo_FootPrint:rkd_cutdot_no_edgecut_4, F.Cu at (83.3, 93.2)
- added REF**: rkd_cutdot_no_edgecut_1, Rikkodo_FootPrint:rkd_cutdot_no_edgecut_1, F.Cu at (75.6, 59.2)
- added REF**: rkd_cutdot_no_edgecut_1, Rikkodo_FootPrint:rkd_cutdot_no_edgecut_1, F.Cu at (88.7, 59.2)
- added REF**: rkd_cutdot_no_edgecut_1, Rikkodo_FootPrint:rkd_cutdot_no_edgecut_1, F.Cu at (93.2, 92.3)
- added REF**: rkd_cutdot_no_edgecut_1, Rikkodo_FootPrint:rkd_cutdot_no_edgecut_1, F.Cu at (88.4, 58.3)
- added REF**: rkd_cutdot_no_edgecut_1, Rikkodo_FootPrint:rkd_cutdot_no_edgecut_1, F.Cu at (91.1, 59.2)
- added REF**: rkd_cutdot_no_edgecut_1, Rikkodo_FootPrint:rkd_cutdot_no_edgecut_1, F.Cu at (88.4, 57.1)
- added REF**: rkd_cutdot_no_edgecut_1, Rikkodo_FootPrint:rkd_cutdot_no_edgecut_1, F.Cu at (93.2, 55.4)
- added REF**: rkd_cutdot_no_edgecut_1, Rikkodo_FootPrint:rkd_cutdot_no_edgecut_1, F.Cu at (94.1, 73.5)
- added REF**: rkd_cutdot_no_edgecut_1, Rikkodo_FootPrint:rkd_cutdot_no_edgecut_1, F.Cu at (74.4, 59.2)
- added REF**: rkd_cutdot_no_edgecut_1, Rikkodo_FootPrint:rkd_cutdot_no_edgecut_1, F.Cu at (88.4, 56.0)
Other:
- board size 57.7 x 38.7 mm -> 57.7 x 39.3 mm
