File: RKD_09/RKD09_Assmenble/RKD09_Assmenble.kicad_pcb (KiCad board)
At the start: 2 copper layers, 57.7 x 39.3 mm, 61 parts, among them J1 Conn_01x06, J3 Qwiic_RA, SW1 SW_Push, SW2 KEY_SWITCH, U1 ProMicro

Commit message: edit Meishi
Parts:
- removed the LED1 at (83.3, 83.3)
- SW1: value SW_Push -> RotaryEncoder_Switch; footprint kbd_SW:CherryMX_Solder_1u -> BrownSugar_KBD:RotaryEncoder_EC11-Switch
- SW2: value KEY_SWITCH -> RotaryEncoder_Switch; footprint kbd_SW_Hole:SW_Hole_1u -> BrownSugar_KBD:RotaryEncoder_EC11-Hole
- turned SW2 to 90 degrees
- renumbered LED2 to LED1
Connections:
- LED1 pad 3: Net-(LED1-DOUT) -> LED
- U1 pad 1: GND -> RE_A
- U1 pad 2: GND -> RE_B
Routing:
- net RE_A: track 0.00 -> 13.5 mm
- net GND: track 93.5 -> 81.6 mm
- net LED: track 6.25 -> 18.0 mm
- net VCC: track 63.2 -> 51.9 mm
- net Net-(LED1-DOUT): track 9.21 -> 0.00 mm
- net RE_B: track 0.00 -> 6.31 mm
- net SDA: track 29.3 -> 31.6 mm
- net SCL: track 26.6 -> 28.2 mm
- net KEY1: track 6.13 -> 6.97 mm
Other:
- board text added: "D2"
- board text added: "D3"
- board text added: "RE_A"
- board text added: "RE_B"
