File: RKD_07/Botsu/RKD07_RePicot_B1/RKD07_RePicot.kicad_sch (KiCad schematic)
At the start: 13 parts, among them J1 Conn_01x06, J2 Conn_01x24, J3 Qwiic_RA, J4 Conn_01x06, J5 Conn_01x02_Socket, J6 Conn_01x06, J8 Conn_01x06, SW41 SW_Push, U1 Pico

Commit message: RemakeRepicot
Parts:
- removed D41: D, kbd_Parts:Diode_SMD, symbol Device:D
- removed J1: Conn_01x06, Connector_PinHeader_2.54mm:PinHeader_1x06_P2.54mm_Horizontal, symbol Connector_Generic:Conn_01x06
- removed J6: Conn_01x06, Connector_Harwin:Harwin_M20-89006xx_1x06_P2.54mm_Horizontal, symbol Connector_Generic:Conn_01x06
- removed SW41: SW_Push, Rikkodo_FootPrint:rkd_Asm_ChocV1V2_Hotswap_1u, symbol Switch:SW_Push
- added J1: TRRS, BrownSugar_KBD:TRRS_PJ-320A, symbol BrownSugar_KBD:TRRS
- added J13, J7, J9: Conn_01x04, Connector_PinHeader_2.54mm:PinHeader_1x04_P2.54mm_Horizontal, symbol Connector_Generic:Conn_01x04
- added R1, R2: 1kΩ, Resistor_THT:R_Axial_DIN0207_L6.3mm_D2.5mm_P10.16mm_Horizontal, symbol Device:R
- J5: footprint Connector_PinHeader_2.54mm:PinHeader_1x02_P2.54mm_Vertical -> Connector_PinHeader_2.54mm:PinHeader_1x02_P2.54mm_Horizontal
- renumbered R1 to R3, R2 to R4
Connections:
- net 3V3: now also R1.1, R2.1
- net COL13_L: now also U1.5 (GPIO3); no longer U1.2 (GPIO1)
- net GND: now also U1.13 (GND), U1.8 (GND), J1.A, J13.4 (Pin_4), J7.4 (Pin_4), J9.1 (Pin_1)
- net SCL/TX_L: now also J13.2 (Pin_2), R1.2
- net SDA/SCK_L: now also J13.3 (Pin_3), R2.2
- net VCC: now also J1.D, J13.1 (Pin_1), J7.1 (Pin_1), J9.4 (Pin_4)
- net GP00_MISO renamed CS
- net CS: now also J9.2 (Pin_2); no longer U1.1 (GPIO0)
- net GP02_SCLK renamed GP01:UART_RX
- net GP01:UART_RX: now also U1.2 (GPIO1), J1.C, J7.3 (Pin_3); no longer U1.4 (GPIO2)
- net GP03_MOSI renamed GP00:UART_TX
- net GP00:UART_TX: now also U1.1 (GPIO0), J1.B, J7.2 (Pin_2); no longer U1.5 (GPIO3)
- new net GP02: J9.3 (Pin_3), U1.4 (GPIO2)
- no-connect marks 14 -> 11
Other:
- note added: "CS"
- note added: "HandDetect"
- note added: "HandDetect And fix nCS"
- note added: "MOTION"
- note removed: "3V3 CS MOTION SDIO SCLK GND"
- note removed: "GND GND GP00_MISO GP02_SCLK GP03_MOSI"
- note removed: "Rabit"
- note removed: "SPI_SMD"
- note removed: "SPI_TH"
- moved on the sheet: J5, J8, OL1
