File: RKD_11/RKD11_Assmenble/RKD11_Assmenble.kicad_pcb (KiCad board)
At the start: 2 copper layers, 58.3 x 39.3 mm, 35 parts, among them J1 Conn_01x06, J3 Qwiic_RA, SW1 RotaryEncoder_Switch, SW2 SW_Push, SW99 KEY_SWITCH, U1 ProMicro

Commit message: Update
Parts:
- removed the REF** at (83.3, 93.2)
- added REF**: rkd_cutdot, Rikkodo_FootPrint:rkd_cutdot, F.Cu at (83.3, 53.9)
Other:
- outline, holes or cut-outs redrawn
Changed lines of the file:
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@@
 		(embedded_fonts no)
 	)
+	(footprint "Rikkodo_FootPrint:rkd_cutdot"
+		(layer "F.Cu")
+		(at 83.34375 53.875736)
+		(property "Reference" "REF**"
+			(at 0 -0.5 0)
+			(unlocked yes)
+			(layer "F.SilkS")
+			(hide yes)
+			(effects
+				(font
+					(size 1 1)
+					(thickness 0.1)
+				)
+			)
+		)
+		(property "Value" "rkd_cutdot"
+			(at 0 1 0)
+			(unlocked yes)
+			(layer "F.Fab")
+			(hide yes)
+			(effects
+				(font
+					(size 1 1)
+					(thickness 0.15)
+				)
+			)
+		)
+		(property "Datasheet" ""
+			(at 0 0 0)
+			(unlocked yes)
+			(layer "F.Fab")
+			(hide yes)
+			(effects
+				(font
+					(size 1 1)
+					(thickness 0.15)
+				)
+			)
+		)
+		(property "Description" ""
+			(at 0 0 0)
+			(unlocked yes)
+			(layer "F.Fab")
+			(hide yes)
+			(effects
+				(font
+					(size 1 1)
+					(thickness 0.15)
+				)
+			)
+		)
+		(attr smd board_only exclude_from_pos_files exclude_from_bom)
+		(fp_line
+			(start 1.190622 0.297656)
+			(end -1.190628 0.297656)
+			(stroke
+				(width 0.05)
+				(type default)
+			)
+			(layer "B.SilkS")
+		)
+		(fp_line
+			(start 1.190623 -0.297657)
+			(end -1.190627 -0.297657)
+			(stroke
+				(width 0.05)
+				(type default)
+			)
+			(layer "B.SilkS")
+		)
+		(fp_line
+			(start -1.190628 0.297656)
+			(end -1.190768 -0.297479)
+			(stroke
+				(width 0.05)
+				(type default)
+			)
+			(layer "Edge.Cuts")
+		)
+		(fp_line
+			(start 1.190624 0.297656)
+			(end 1.190482 -0.297479)
+			(stroke
+				(width 0.05)
+				(type default)
+			)
+			(layer "Edge.Cuts")
+		)
+		(pad "" np_thru_hole circle
+			(at -0.893198 0.000356 90)
+			(size 0.5 0.5)
+			(drill 0.5)
+			(layers "*.Cu" "*.Mask")
+		)
+		(pad "" np_thru_hole circle
+			(at -0.297886 0.000356 90)
+			(size 0.5 0.5)
+			(drill 0.5)
+			(layers "*.Cu" "*.Mask")
+		)
+		(pad "" np_thru_hole circle
+			(at 0.297426 0.000356 90)
+			(size 0.5 0.5)
+			(drill 0.5)
+			(layers "*.Cu" "*.Mask")
+		)
+		(pad "" np_thru_hole circle
+			(at 0.892738 0.000356 90)
+			(size 0.5 0.5)
+			(drill 0.5)
+			(layers "*.Cu" "*.Mask")
+		)
+		(embedded_fonts no)
+	)
 	(footprint "kbd_Hole:m2_Screw_Hole"
 		(layer "F.Cu")
@@
 		(embedded_fonts no)
 	)
-	(footprint "Rikkodo_FootPrint:rkd_cutdot_no_edgecut_4"
-		(layer "F.Cu")
-		(at 83.343909 93.165617)
-		(property "Reference" "REF**"
-			(at 0 -0.5 0)
-			(unlocked yes)
-			(layer "F.SilkS")
-			(hide yes)
-			(effects
-				(font
-					(size 1 1)
-					(thickness 0.1)
-				)
-			)
-		)
-		(property "Value" "rkd_cutdot_no_edgecut_4"
-			(at 0 1 0)
-			(unlocked yes)
-			(layer "F.Fab")
-			(hide yes)
-			(effects
-				(font
-					(size 1 1)
-					(thickness 0.15)
-				)
-			)
-		)
-		(property "Datasheet" ""
-			(at 0 0 0)
-			(unlocked yes)
-			(layer "F.Fab")
-			(hide yes)
-			(effects
-				(font
-					(size 1 1)
-					(thickness 0.15)
-				)
-			)
-		)
-		(property "Description" ""
-			(at 0 0 0)
-			(unlocked yes)
-			(layer "F.Fab")
-			(hide yes)
-			(effects
-				(font
-					(size 1 1)
-					(thickness 0.15)
-				)
-			)
-		)
-		(attr smd board_only exclude_from_pos_files exclude_from_bom)
-		(fp_line
-			(start -0.000001 0.298011)
-			(end -2.381251 0.298011)
-			(stroke
-				(width 0.05)
-				(type default)
-			)
-			(layer "B.SilkS")
-		)
-		(fp_line
-			(start 0 -0.297302)
-			(end -2.38125 -0.297302)
-			(stroke
-				(width 0.05)
-				(type default)
-			)
-			(layer "B.SilkS")
-		)
-		(fp_line
-			(start 2.381249 0.298012)
-			(end -0.000001 0.298012)
-			(stroke
-				(width 0.05)
-				(type default)
-			)
-			(layer "B.SilkS")
-		)
-		(fp_line
-			(start 2.38125 -0.297301)
-			(end 0 -0.297301)
-			(stroke
-				(width 0.05)
-				(type default)
-			)
-			(layer "B.SilkS")
-		)
-		(pad "" np_thru_hole circle
-			(at -2.083821 0.000711 90)
-			(size 0.5 0.5)
-			(drill 0.5)
-			(layers "*.Cu" "*.Mask")
-		)
-		(pad "" np_thru_hole circle
-			(at -1.488509 0.000711 90)
-			(size 0.5 0.5)
-			(drill 0.5)
-			(layers "*.Cu" "*.Mask")
-		)
-		(pad "" np_thru_hole circle
-			(at -0.893197 0.000711 90)
-			(size 0.5 0.5)
-			(drill 0.5)
-			(layers "*.Cu" "*.Mask")
-		)
-		(pad "" np_thru_hole circle
-			(at -0.297885 0.000711 90)
-			(size 0.5 0.5)
-			(drill 0.5)
-			(layers "*.Cu" "*.Mask")
-		)
-		(pad "" np_thru_hole circle
-			(at 0.297429 0.000712 90)
-			(size 0.5 0.5)
-			(drill 0.5)
-			(layers "*.Cu" "*.Mask")
-		)
-		(pad "" np_thru_hole circle
-			(at 0.892741 0.000712 90)
-			(size 0.5 0.5)
-			(drill 0.5)
-			(layers "*.Cu" "*.Mask")
-		)
-		(pad "" np_thru_hole circle
-			(at 1.488053 0.000712 90)
-			(size 0.5 0.5)
-			(drill 0.5)
-			(layers "*.Cu" "*.Mask")
-		)
-		(pad "" np_thru_hole circle
-			(at 2.083365 0.000712 90)
-			(size 0.5 0.5)
-			(drill 0.5)
-			(layers "*.Cu" "*.Mask")
-		)
-		(embedded_fonts no)
-	)
 	(footprint "kbd_Hole:m2_Screw_Hole"
 		(layer "F.Cu")
@@
 	)
 	(gr_line
-		(start 113.109192 55.364236)
-		(end 113.109193 91.678268)
+		(start 93.463983 54.173392)
+		(end 93.463984 92.868672)
 		(stroke
 			(width 0.05)
 			(type solid)
 		)
-		(layer "B.SilkS")
+		(layer "F.SilkS")
 	)
-	(gr_arc
-		(start 92.86875 91.678125)
-		(mid 92.520017 92.520017)
-		(end 91.678125 92.86875)
+	(gr_line
+		(start 113.10928 54.173392)
+		(end 113.109281 92.868672)
+		(stroke
+			(width 0.05)
+			(type solid)
+		)
+		(layer "F.SilkS")
+	)
+	(gr_line
+		(start 92.868671 54.173392)
+		(end 92.868672 92.868672)
+		(stroke
+			(width 0.05)
+			(type solid)
+		)
+		(layer "F.SilkS")
+	)
+	(gr_line
+		(start 112.513968 54.173392)
+		(end 112.513969 92.868672)
+		(stroke
+			(width 0.05)
+			(type solid)
+		)
+		(layer "F.SilkS")
+	)
+	(gr_line
+		(start 113.109192 55.364236)
+		(end 113.109193 91.678268)
 		(stroke
 			(width 0.05)
@@
 	)
 	(gr_arc
-		(start 94.6546 92.857489)
-		(mid 93.8163 92.512423)
-		(end 93.463984 91.677148)
+		(start 92.86875 91.678125)
+		(mid 92.520017 92.520017)
+		(end 91.678125 92.86875)
 		(stroke
 			(width 0.05)
@@
 		(layer "B.SilkS")
 	)
+	(gr_arc
+		(start 94.654608 92.868622)
+		(mid 93.812775 92.519941)
+		(end 93.464034 91.678132)
+		(stroke
+			(width 0.05)
+			(type solid)
+		)
+		(layer "B.SilkS")
+	)
 	(gr_line
 		(start 93.464033 55.3641)
@@
 	(gr_line
 		(start 91.6781 92.86875)
-		(end 85.724928 92.868637)
-		(stroke
-			(width 0.05)
-			(type default)
-		)
-		(layer "Edge.Cuts")
-	)
-	(gr_line
-		(start 85.724928 93.463984)
-		(end 85.724928 92.868637)
+		(end 74.711718 92.868428)
 		(stroke
 			(width 0.05)
@@
 	)
 	(gr_line
-		(start 80.962432 93.463984)
-		(end 85.724928 93.463984)
-		(stroke
-			(width 0.05)
-			(type default)
-		)
-		(layer "Edge.Cuts")
-	)
-	(gr_line
-		(start 80.962432 92.868672)
-		(end 80.962432 93.463984)
+		(start 84.534373 53.578079)
+		(end 82.152982 53.578257)
 		(stroke
 			(width 0.05)
@@
 	(gr_line
 		(start 91.678048 54.173393)
-		(end 74.711656 54.173392)
+		(end 84.534374 54.173392)
 		(stroke
 			(width 0.05)
@@
 	(gr_line
 		(start 91.6781 92.869914)
-		(end 94.6546 92.857489)
+		(end 94.6545 92.868672)
 		(stroke
 			(width 0.05)
@@
 	)
 	(gr_line
-		(start 94.6545 92.857489)
+		(start 94.6545 92.868672)
 		(end 111.323373 92.857297)
 		(stroke
@@
 	)
 	(gr_line
-		(start 80.962432 92.868672)
-		(end 74.711718 92.868749)
+		(start 82.153122 54.173392)
+		(end 74.711656 54.173389)
 		(stroke
 			(width 0.05)
@@
 		(polygon
 			(pts
-				(xy 73.818532 59.828856) (xy 78.283372 59.828856) (xy 78.283372 54.173483) (xy 87.213052 54.173483)
-				(xy 87.213052 59.828856) (xy 92.27336 59.828856) (xy 92.27336 92.868828) (xy 73.818532 92.868828)
+				(xy 74.414 59.828856) (xy 78.87884 59.828856) (xy 78.87884 54.768704) (xy 87.80852 54.768704) (xy 87.80852 59.828856)
+				(xy 92.27336 59.828856) (xy 92.27336 92.868828) (xy 74.414 92.868828)
 			)
 		)
