File: RKD_07_RE/RKD07_RePicotSplitHead/RKD07_RePicotSplitHead.kicad_pcb (KiCad board)
At the start: 2 copper layers, 61.3 x 98.2 mm, 16 parts, among them J101 Conn_01x24, J102 Conn_01x06, J151 Conn_01x06, J152 RJ9, J153 TRRS, J154 Conn_01x02_Socket, J155 Conn_01x02_Socket, J156 Conn_01x02_Socket, U101 Pico

Commit message: ModifyDots
Parts:
- added Ref**: Val**, kbd_Hole:m2_Screw_Hole, F.Cu at (81.0, 56.0)
- added Ref**: Val**, kbd_Hole:m2_Screw_Hole, F.Cu at (81.0, 108.3)
- added Ref**: Val**, kbd_Hole:m2_Screw_Hole, F.Cu at (83.3, 36.9)
Routing:
- net GND: track 122.4 -> 126.9 mm, vias 13 -> 17
- net COL13_L: track 13.7 -> 18.2 mm
- net GP04: track 124.5 -> 121.5 mm
- net ROW0_L: track 25.8 -> 24.0 mm
- net GP07: track 144.1 -> 143.0 mm
- net GP02_SCLK: track 64.6 -> 63.7 mm
- net GP01_NCS: track 58.6 -> 59.3 mm
Other:
- board size 61.3 x 98.2 mm -> 61.3 x 82.7 mm
