File: RKD_07_SP/RKD07_RePicotSmallBody/RKD07_RePicotSmallBody.kicad_pcb (KiCad board)
At the start: 2 copper layers, 36.9 x 36.9 mm, 19 parts, among them J201 Conn_01x06, J251 Conn_01x02_Socket, J252 Conn_01x06, J253 Conn_01x02_Socket, J254 Conn_01x02_Socket, U201 TLV70019DDCR, U202 PMW3610DM-SUDU

Commit message: RePicotUpdate
Parts:
- moved J252 1.19 mm to (133.2, 63.1)
Routing:
- net 3V3_E: track 68.1 -> 94.6 mm, vias 2 -> 0
- net GP03_MOSI_E: track 34.2 -> 30.8 mm
- net GND_E: track 118.4 -> 116.6 mm, vias 9 -> 12
- net GP00_MISO_E: track 33.2 -> 31.4 mm
- net GP02_SCLK_E: track 35.0 -> 33.4 mm
- net NCS_E: track 71.2 -> 71.5 mm, vias 3 -> 0
Other:
- board text added: "0.01u"
- board text added: "0.1u"
- board text added: "10u"
- board text added: "1u"
- board text added: "3.3u"
- board text added: "3V3 NCS SDIO SCLK MOTN GND"
- board text removed: "0.01uF"
- board text removed: "0.1uF"
- board text removed: "10uF"
- board text removed: "1uF"
- board text removed: "3.3uF"
