File: RKD_07_Zwei/RKD07_Assemble_ZWEI/RKD07_Assemble_ZWEI.kicad_sch (KiCad schematic)
At the start: 178 parts, among them J1 Conn_01x24, J2 Conn_01x24, J21 Conn_01x02_Socket, J22 Conn_01x02_Socket, J23 Conn_01x10, J24 Conn_01x06, J3 Conn_01x12, J4 Conn_01x06, J51 RJ12, J52 RJ12, J53 Qwiic_RA, J6 Conn_01x06, J7 Conn_01x06, J8 Conn_01x12, SW1 SW_Push, SW10 SW_Push, SW11 SW_Push, SW12 SW_Push, SW13 SW_Push, SW14 SW_Push, SW15 SW_Push, SW16 SW_Push, SW17 SW_Push, SW18 SW_Push, SW19 SW_Push, SW2 SW_Push, SW20 SW_Push, SW21 SW_Push, SW22 SW_Push, SW23 SW_Push, SW24 SW_Push, SW25 SW_Push, SW26 SW_Push, SW27 SW_Push, SW28 SW_Push, SW29 SW_Push, SW3 SW_Push, SW30 RotaryEncoder_Switch, SW31 SW_Push, SW4 SW_Push, SW49 RotaryEncoder_Switch, SW5 SW_Push, SW50 SW_Push, SW51 SW_Push, SW52 SW_Push, SW53 SW_Push, SW54 SW_Push, SW55 SW_Push, SW56 SW_Push, SW57 SW_Push, SW58 SW_Push, SW59 SW_Push, SW6 SW_Push, SW60 SW_Push, SW61 SW_Push, SW62 SW_Push, SW63 SW_Push, SW64 SW_Push, SW65 SW_Push, SW66 SW_Push, SW67 SW_Push, SW68 SW_Push, SW69 SW_Push, SW7 SW_Push, SW70 SW_Push, SW71 SW_Push, SW72 SW_Push, SW73 SW_Push, SW74 SW_Push, SW75 SW_Push, SW76 SW_Push, SW77 SW_Push, SW78 SW_Push, SW79 SW_Push, SW8 SW_Push, SW80 SW_Push, SW81 SW_Push, SW82 SW_Push, SW83 SW_Push, SW84 SW_Push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

Commit message: ZWEI_TOP/BOTTOM
Parts:
- added SW32: SW_Push, Rikkodo_FootPrint:rkd_Asm_ChocV1V2_Hotswap_1u_NM, symbol Switch:SW_Push
Connections:
- net COL10_L: now also SW32.1
- net at D31.2 (A), SW31.1: now also SW32.2
Changed lines of the file:
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@@
 	)
 	(junction
+		(at 196.85 246.38)
+		(diameter 0)
+		(color 0 0 0 0)
+	)
+	(junction
 		(at 521.97 250.19)
 		(diameter 0)
@@
 	(wire
 		(pts
+			(xy 196.85 228.6) (xy 196.85 246.38)
+		)
+		(stroke
+			(width 0)
+			(type default)
+		)
+	)
+	(wire
+		(pts
 			(xy 608.33 308.61) (xy 633.73 308.61)
 		)
@@
 		)
 	)
+	(global_label "COL10_L"
+		(shape input)
+		(at 186.69 228.6 180)
+		(fields_autoplaced yes)
+		(effects
+			(font
+				(size 1.27 1.27)
+			)
+			(justify right)
+		)
+		(property "Intersheetrefs" "${INTERSHEET_REFS}"
+			(at 175.6615 228.6 0)
+			(effects
+				(font
+					(size 1.27 1.27)
+				)
+				(justify right)
+				(hide yes)
+			)
+		)
+	)
 	(global_label "COL1_GP16_R"
 		(shape input)
@@
 					(unit 1)
 				)
+			)
+		)
+	)
+	(symbol
+		(lib_id "Switch:SW_Push")
+		(at 191.77 228.6 0)
+		(unit 1)
+		(exclude_from_sim no)
+		(in_bom yes)
+		(on_board yes)
+		(dnp no)
+		(fields_autoplaced yes)
+		(property "Reference" "SW32"
+			(at 191.77 220.98 0)
+			(effects
+				(font
+					(size 1.27 1.27)
+				)
+			)
+		)
+		(property "Value" "SW_Push"
+			(at 191.77 223.52 0)
+			(effects
+				(font
+					(size 1.27 1.27)
+				)
+			)
+		)
+		(property "Footprint" "Rikkodo_FootPrint:rkd_Asm_ChocV1V2_Hotswap_1u_NM"
+			(at 191.77 223.52 0)
+			(effects
+				(font
+					(size 1.27 1.27)
+				)
+				(hide yes)
+			)
+		)
+		(property "Datasheet" "~"
+			(at 191.77 223.52 0)
+			(effects
+				(font
+					(size 1.27 1.27)
+				)
+				(hide yes)
+			)
+		)
+		(property "Description" "Push button switch, generic, two pins"
+			(at 191.77 228.6 0)
+			(effects
+				(font
+					(size 1.27 1.27)
+				)
+				(hide yes)
+			)
+		)
+		(pin "1"
+		)
+		(pin "2"
+		)
+		(instances
+			(project "RKD07_Assemble_ZWEI"
+				(path "/01a859e0-5a12-4534-b9e3-6128f69eb8fc"
+					(reference "SW32")
+					(unit 1)
+				)

Commit message: update
Parts:
- added J5: Conn_01x06, Connector_FFC-FPC:Hirose_FH12-6S-0.5SH_1x06-1MP_P0.50mm_Horizontal, symbol Connector_Generic:Conn_01x06
- added J9: Conn_01x06, Connector_PinHeader_2.54mm:PinHeader_1x06_P2.54mm_Vertical, symbol Connector_Generic:Conn_01x06
Connections:
- net 3v3_R: now also J5.6 (Pin_6), J9.6 (Pin_6)
- net GND_R: now also J5.1 (Pin_1), J5.5 (Pin_5), J9.1 (Pin_1), J9.2 (Pin_2)
- net GP00_R: now also J5.4 (Pin_4), J9.3 (Pin_3)
- net GP02_R: now also J5.3 (Pin_3), J9.4 (Pin_4)
- net GP03_R: now also J5.2 (Pin_2), J9.5 (Pin_5)
Other:
- note added: "GND GND GP00_MISO GP02_SCLK GP03_MOSI"
- note added: "Nogikesuya_TrackBall"
- note added: "SPI_TH"
