File: RKD_12/RKD12_ASM/RKD12_ASM.kicad_pcb (KiCad board)
At the start: 2 copper layers, 98.8 x 97.7 mm, 48 parts, among them J1 Conn_01x24, J51 Conn_01x06, J52 Qwiic_RA, J53 RJ9, J54 Conn_01x02_Socket, J6 Conn_01x12, SW1 SW_Push, SW10 SW_Push, SW11 SW_Push, SW12 SW_Push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

Commit message: update
Parts:
- added J2: Conn_01x06, Connector_FFC-FPC:Hirose_FH12-6S-0.5SH_1x06-1MP_P0.50mm_Horizontal, B.Cu at (87.7, 49.3)
- added Ref**: Val**, kbd_Hole:m2_Spacer_Hole_hex, F.Cu at (121.4, 83.3)
- added Ref**: Val**, kbd_Hole:m2_Spacer_Hole_hex, F.Cu at (159.5, 83.3)
- added Ref**: Val**, kbd_Hole:m2_Spacer_Hole_hex, F.Cu at (140.5, 45.2)
- added SW19: SW_Push, kbd_Parts:ResetSW, F.Cu at (100.6, 96.1)
- J53: value RJ9 -> 6P6C; footprint Connector_RJ:RJ9_Evercom_5301-440xxx_Horizontal -> Connector_RJ:RJ12_Amphenol_54601-x06_Horizontal
- moved J53 2.93 mm to (98.3, 92.1)
- moved SW5 2.38 mm to (90.5, 111.9)
- moved D5 1.19 mm to (85.1, 106.0)
- moved J54 0.98 mm to (95.3, 53.0)
- renumbered J6 to J3
Connections:
- J1 pad 5: COL13_R -> GP01_NCS_COL13_R
- J51 pad 2: GND_R -> GP01_NCS_COL13_R
- J53 pad 1: GND_R -> unconnected-(J53-Pad1)
- J53 pad 2: COL1_GP16_R -> GND_R
- J53 pad 3: COL0_GP17_R -> COL1_GP16_R
- J53 pad 4: VCC_R -> COL0_GP17_R
- U1 pad 2: COL13_R -> GP01_NCS_COL13_R
Routing:
- net GP01_NCS_COL13_R: track 0.00 -> 50.3 mm
- net COL13_R: track 44.7 -> 0.00 mm
- net 3V3_R: track 82.5 -> 118.8 mm
- net GND_R: track 258.5 -> 280.1 mm, vias 31 -> 35
- net GP00_MISO_R: track 12.2 -> 32.0 mm
- net GP02_SCLK_R: track 10.1 -> 29.6 mm
- net Net-(D5-A): track 9.52 -> 24.2 mm
- net GP03_MOSI_R: track 7.15 -> 21.8 mm
- net SDA/SCK_R: track 60.1 -> 52.0 mm
- net COL1_GP16_R: track 110.2 -> 114.2 mm
- net ROW3_R: track 136.7 -> 133.3 mm
- net GP07_RE_B_R: track 87.2 -> 90.6 mm
- net GP04_RE_A_R: track 103.4 -> 100.7 mm
- net ROW4_R: track 123.9 -> 126.6 mm
- net COL5_R: track 306.9 -> 309.4 mm
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Other:
- outline, holes or cut-outs redrawn
- board text added: "JLCJLCJLC"
- board text added: "Nogi"
- board text added: "RKD12_Asm_v1.0"

Commit message: update
Parts:
- added J4: Conn_01x06, DreaM117er-keebLibrary:Hirose_FH12-6S-0.5SH_1x06-1MP_P0.50mm_Horizontal, B.Cu at (120.6, 49.2)
- added R1: 1kΩ, Resistor_SMD:R_0603_1608Metric, B.Cu at (96.1, 89.0)
- added R2: 1kΩ, Resistor_SMD:R_0603_1608Metric, B.Cu at (96.1, 87.2)
Routing:
- net COL7_R: track 24.7 -> 91.0 mm, vias 0 -> 1
- net COL6_R: track 18.5 -> 69.1 mm, vias 0 -> 2
- net GP07_RE_B_R: track 90.6 -> 130.5 mm, vias 0 -> 1
- net GP04_RE_A_R: track 100.7 -> 137.9 mm, vias 0 -> 1
- net COL10_R: track 16.2 -> 42.1 mm, vias 0 -> 1
- net GND_R: track 280.1 -> 299.1 mm, vias 35 -> 36
- net 3V3_R: track 118.8 -> 123.8 mm
- net SDA/SCK_R: track 52.0 -> 55.5 mm
- net SCL/TX_R: track 65.3 -> 68.6 mm
- net ROW1_R: track 142.4 -> 145.8 mm
- net VCC_R: track 110.0 -> 111.2 mm
- net COL3_R: track 183.1 -> 184.1 mm
- net COL4_R: track 168.5 -> 169.4 mm
- net COL2_R: track 187.7 -> 188.6 mm
- net COL0_GP17_R: track 109.6 -> 108.8 mm
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
Commit message: modify
Routing:
- net ROW4_R: track 127.2 -> 130.6 mm
- net GP07_RE_B_R: track 130.5 -> 131.9 mm
- net GND_R: vias 36 -> 37
Changed lines of the file:
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@@
 	)
 	(via
-		(at 105.965625 46.434375)
+		(at 105.965625 45.839101)
 		(size 0.6)
 		(drill 0.3)
@@
 	)
 	(via
+		(at 111.323531 45.839101)
+		(size 0.6)
+		(drill 0.3)
+		(layers "F.Cu" "B.Cu")
+		(free yes)
+		(net 13)
+	)
+	(via
 		(at 170.259375 120.253125)
 		(size 0.6)
@@
 	)
 	(segment
+		(start 84.848827 118.190681)
+		(end 87.427897 120.76975)
+		(width 0.3)
+		(layer "F.Cu")
+		(net 32)
+	)
+	(segment
+		(start 82.490392 51.1175)
+		(end 80.4615 53.146392)
+		(width 0.3)
+		(layer "F.Cu")
+		(net 32)
+	)
+	(segment
 		(start 91.6365 120.76975)
 		(end 92.9875 119.41875)
@@
 	)
 	(segment
+		(start 80.4615 53.146392)
+		(end 80.4615 116.18028)
+		(width 0.3)
+		(layer "F.Cu")
+		(net 32)
+	)
+	(segment
 		(start 93.995454 54.183857)
 		(end 96.430079 54.183857)
@@
 	)
 	(segment
+		(start 84.093518 118.190681)
+		(end 84.848827 118.190681)
+		(width 0.3)
+		(layer "F.Cu")
+		(net 32)
+	)
+	(segment
 		(start 118.853548 47.2385)
 		(end 119.955368 46.13668)
@@
 	)
 	(segment
-		(start 80.4615 53.146392)
-		(end 80.4615 113.803353)
+		(start 83.101383 117.198546)
+		(end 84.093518 118.190681)
+		(width 0.3)
+		(layer "F.Cu")
+		(net 32)
+	)
+	(segment
+		(start 80.4615 116.18028)
+		(end 81.479766 117.198546)
 		(width 0.3)
 		(layer "F.Cu")
@@
 	)
 	(segment
-		(start 98.568392 48.581029)
-		(end 99.910921 47.2385)
+		(start 81.479766 117.198546)
+		(end 83.101383 117.198546)
 		(width 0.3)
 		(layer "F.Cu")
@@
 	)
 	(segment
-		(start 87.427897 120.76975)
-		(end 91.6365 120.76975)
+		(start 98.568392 48.581029)
+		(end 99.910921 47.2385)
 		(width 0.3)
 		(layer "F.Cu")
@@
 	)
 	(segment
-		(start 80.4615 113.803353)
-		(end 87.427897 120.76975)
+		(start 87.427897 120.76975)
+		(end 91.6365 120.76975)
 		(width 0.3)
 		(layer "F.Cu")
@@
 	)
 	(segment
-		(start 82.490392 51.1175)
-		(end 80.4615 53.146392)
-		(width 0.3)
-		(layer "F.Cu")
-		(net 32)
-	)
-	(segment
 		(start 96.430079 54.183857)
 		(end 98.568392 52.045544)
@@
 	)
 	(segment
-		(start 92.9875 104.91875)
-		(end 100.607897 97.298353)
+		(start 99.3685 94.108225)
+		(end 99.3685 98.53775)
 		(width 0.3)
 		(layer "F.Cu")
@@
 	)
 	(segment
-		(start 100.607897 97.298353)
-		(end 100.607897 92.868828)
+		(start 99.3685 98.53775)
+		(end 92.9875 104.91875)
+		(width 0.3)
+		(layer "F.Cu")
+		(net 36)
+	)
+	(segment
+		(start 100.607897 92.868828)
+		(end 99.3685 94.108225)
 		(width 0.3)
 		(layer "F.Cu")
@@
 	)
 	(segment
+		(start 101.503691 39.591191)
+		(end 101.503691 42.2642)
+		(width 0.3)
+		(layer "F.Cu")
+		(net 50)
+	)
+	(segment
 		(start 128.5875 32.146875)
 		(end 147.6375 32.146875)
@@
 	)
 	(segment
+		(start 101.503691 42.2642)
+		(end 100.270392 43.4975)
+		(width 0.3)
+		(layer "F.Cu")
+		(net 50)
+	)
+	(segment
 		(start 147.6375 32.146875)
 		(end 164.30625 32.146875)
@@
 	)
 	(segment
-		(start 100.270392 43.4975)
-		(end 104.179775 39.588117)
+		(start 104.179775 36.91511)
+		(end 101.503691 39.591191)
 		(width 0.3)
 		(layer "F.Cu")
@@
 	)
 	(segment
-		(start 104.179775 34.855725)
-		(end 106.877659 32.157841)
+		(start 106.877659 32.157841)
+		(end 106.888625 32.146875)
 		(width 0.3)
 		(layer "F.Cu")
@@
 	)
 	(segment
-		(start 104.179775 39.588117)
-		(end 104.179775 34.855725)
+		(start 104.179775 34.855725)
+		(end 104.179775 36.91511)
 		(width 0.3)
 		(layer "F.Cu")
@@
 	(segment
 		(start 106.877659 32.157841)
-		(end 106.888625 32.146875)
+		(end 104.179775 34.855725)
 		(width 0.3)
 		(layer "F.Cu")
@@
 	)
 	(segment
-		(start 132.170384 95.76975)
-		(end 133.86975 94.070384)
-		(width 0.3)
-		(layer "F.Cu")
-		(net 54)
-	)
-	(segment
-		(start 130.693583 95.76975)
-		(end 132.170384 95.76975)
-		(width 0.3)
-		(layer "F.Cu")
-		(net 54)
-	)
-	(segment
-		(start 133.86975 93.269844)
-		(end 142.279807 84.859787)
-		(width 0.3)
-		(layer "F.Cu")
-		(net 54)
-	)
-	(segment
-		(start 133.86975 94.070384)
-		(end 133.86975 93.269844)
-		(width 0.3)
-		(layer "F.Cu")
-		(net 54)
-	)
-	(segment
-		(start 125.435583 101.02775)
-		(end 130.693583 95.76975)
+		(start 142.279807 91.502742)
+		(end 142.279807 67.865682)
 		(width 0.3)
 		(layer "F.Cu")
@@
 	(segment
 		(start 123.229791 101.02775)
-		(end 125.435583 101.02775)
+		(end 132.754799 101.02775)
 		(width 0.3)
 		(layer "F.Cu")
@@
 	)
 	(segment
-		(start 142.279807 84.859787)
-		(end 142.279807 67.865682)
+		(start 132.754799 101.02775)
+		(end 142.279807 91.502742)
 		(width 0.3)
 		(layer "F.Cu")

Commit message: Order1
Other:
- board text removed: "Qwiic"
Changed lines of the file:
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@@
 			(drillshape 0)
 			(scaleselection 1)
-			(outputdirectory "../../../Order/20241231/RKD07/RePicot")
+			(outputdirectory "../../../Order/20241231/RKD12/Asm")
 		)
 	)
@@
 		(layer "B.SilkS")
 		(effects
-			(font
-				(size 1 1)
-				(thickness 0.1)
-			)
-			(justify right bottom mirror)
-		)
-	)
-	(gr_text "Qwiic"
-		(at 276.225307 -6.934461 270)
-		(layer "B.SilkS")
-		(effects

Commit message: Error
Parts:
- moved SW10 1.19 mm to (121.4, 111.9)
- moved SW16 1.19 mm to (169.1, 64.3)
Routing:
- net Net-(D16-A): track 6.32 -> 7.42 mm
Changed lines of the file:
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@@
 	(footprint "Rikkodo_FootPrint:rkd_Asm_ChocV1V2_Hotswap_1u_NM"
 		(layer "F.Cu")
-		(at 122.634375 111.91875 -90)
+		(at 121.44375 111.91875 -90)
 		(property "Reference" "SW10"
 			(at -5.08 -6.35 90)
@@
 		(tags "RJ12 connector")
 		(property "Reference" "J53"
-			(at -1.66 -2.16 270)
+			(at -1.66 -2.16 90)
 			(layer "F.SilkS")
 			(hide yes)
@@
 		)
 		(property "Value" "6P6C"
-			(at 3.55 18.3 270)
+			(at 3.55 18.3 90)
 			(layer "F.Fab")
 			(effects
@@
 	(footprint "Rikkodo_FootPrint:rkd_Asm_ChocV1V2_Hotswap_1u_NM"
 		(layer "F.Cu")
-		(at 169.06875 63.103125)
+		(at 169.06875 64.29375)
 		(property "Reference" "SW16"
 			(at -5.08 -6.35 0)
@@
 	)
 	(segment
-		(start 163.700136 64.889117)
+		(start 164.086931 65.54475)
+		(end 165.497014 64.134667)
+		(width 0.3)
+		(layer "B.Cu")
+		(net 47)
+	)
+	(segment
+		(start 165.497014 64.134667)
 		(end 165.497014 63.092239)
 		(width 0.3)
@@
 	)
 	(segment
-		(start 162.632758 64.889117)
-		(end 163.700136 64.889117)
+		(start 163.16775 65.54475)
+		(end 164.086931 65.54475)
 		(width 0.3)
 		(layer "B.Cu")
@@
 	)
 	(segment
-		(start 160.71875 66.803125)
-		(end 162.632758 64.889117)
+		(start 160.71875 67.99375)
+		(end 163.16775 65.54475)
 		(width 0.3)
 		(layer "B.Cu")

Commit message: update
Changed lines of the file:
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@@
 		(layer "Edge.Cuts")
-	)
-	(gr_text "JLCJLCJLC"
-		(at 114.3 121.44375 0)
-		(layer "F.SilkS")
-		(effects
-			(font
-				(size 1 1)
-				(thickness 0.1)
-			)
-			(justify left bottom)
-		)
-	)
-	(gr_text "RKD12_Asm_v1.0"
-		(at 85.725 121.44375 0)
-		(layer "F.SilkS")
-		(effects
-			(font
-				(size 1 1)
-				(thickness 0.1)
-			)
-			(justify left bottom)
-		)
 	)
 	(gr_text "Nogi\n"
@@
 			)
 			(justify right bottom mirror)
+		)
+	)
+	(gr_text "JLCJLCJLC"
+		(at 122.039165 121.443852 0)
+		(layer "B.SilkS")
+		(effects
+			(font
+				(size 1 1)
+				(thickness 0.1)
+			)
+			(justify left bottom mirror)
 		)
 	)
@@
 		)
 	)
+	(gr_text "RKD12_Asm_v1.0"
+		(at 98.226645 116.086035 0)
+		(layer "B.SilkS")
+		(effects
+			(font
+				(size 1 1)
+				(thickness 0.1)
+			)
+			(justify left bottom mirror)
+		)
+	)
